File: hardware/PS-BPSLeader.kicad_pcb (KiCad board)
At the start: 4 copper layers, 100 x 100 mm, 386 parts, among them IC1 TCAN3413DR, IC2 TCAN3413DR, IC3 CYPD3177-24LQXQ, IC4 BQ79600PWRQ1, IC5 LM74502DDFR, IC6 TCAN3413DR, IC7 TPS552872RYQR, J1 USB_C_Receptacle_USB2.0_16P, J10 Low SIde Conn, J11 SWD_Header, J12 SWD, J13 USB_C_Receptacle_USB2.0_16P, J14 Conn_01x02, J15 Contactor Connector, J16 Contactor Connector, J17 Contactor Connector, J2 ELCON CAN DEBUG, J3 ELCON CAN, J4 Conn_02x06_Counter_Clockwise, J5 CAR CAN IN, J6 CAR CAN OUT, J7 BPS CAN DEBUG, J8 BPS CAN, J9 High Side Conn, Q1 SQ2315CES-T1_GE3, Q10 SI7997DP-T1-GE3, Q11 SI7997DP-T1-GE3, Q12 IRLML0030, Q13 PSMN012-100YS, Q14 PSMN012-100YS, Q2 SQ2315CES-T1_GE3, Q3 SQ2315CES-T1_GE3, Q4 IRLML0030, Q5 IRLML0030, Q6 IRLML0030, Q7 IRLML0030, Q8 IRLML0030, Q9 IRLML0030, SW1 SW_SPDT, SW2 BOOT Switch, SW3 RESET Button, T1 HMU1228NL, T2 HMU1228NL, U1 STM32G473VETx, U10 MCP1826S, U11 TPS2117DRLR, U12 LMR51635XDDCR, U13 PESD5V0L2BT, U14 PESD5V0L2BT, U15 TPS2117DRLR, U16 MCP1826S, U17 TPS2121RUXR, U18 CDSOT23-T24CAN, U2 CDSOT23-T24CAN, U3 CDSOT23-T24CAN, U4 ESP32-C6-MINI-1, U5 DRV110APWR, U6 TPS2121RUXR, U7 DRV110APWR, U8 DRV110APWR, U9 EMC2305-1-AP-TR, Y1 Crystal

Commit message: reviewed
Parts:
- D21: moved to B.Cu
- FAN1, FAN2: footprint Connector_Molex:Molex_Nano-Fit_105309-xx04_1x04_P2.50mm_Vertical -> LHRS_Connectors:Molex_Nano-Fit_105309-xx04_1x04_P2.50mm_Vertical
- moved D22 13.5 mm to (149.8, 41.9), turned to 0 degrees
- moved D21 10.9 mm to (134.6, 45.4), turned to 90 degrees
- moved FAN1 3.11 mm to (141.8, 37.9)
- moved FAN2 1.40 mm to (128.1, 52.1)
Routing:
- net /Fan/FAN_2_PWM: track 9.84 -> 15.5 mm
- net /Fan/FAN_1_TACH: track 15.1 -> 19.4 mm
- net +12V: track 42.3 -> 45.3 mm
- net /Fan/FAN_1_PWM: track 16.1 -> 13.4 mm
- net GND: track 136.1 -> 137.3 mm, vias 211 -> 217
Other:
- board text added: "BPSL Rev A Tony Chen 9/26"
- board text added: "CHARGER CAN"
- board text added: "ELCON FUSE"
- board text added: "ESP BOOT"
- board text added: "ESTOP 2+"
- board text added: "OUT"
- board text added: "PDU_LV+"
- board text added: "STM BOOT"
- board text added: "SWD"
- board text added: "USB PD FUSE"
