File: hardware/PS-BPSLeader.kicad_pcb (KiCad board)
At the start: 4 copper layers, 100 x 100 mm, 386 parts, among them IC1 TCAN3413DR, IC2 TCAN3413DR, IC3 CYPD3177-24LQXQ, IC4 BQ79600PWRQ1, IC5 LM74502DDFR, IC6 TCAN3413DR, IC7 TPS552872RYQR, J1 USB_C_Receptacle_USB2.0_16P, J10 Low SIde Conn, J11 SWD_Header, J12 SWD, J13 USB_C_Receptacle_USB2.0_16P, J14 Conn_01x02, J15 Contactor Connector, J16 Contactor Connector, J17 Contactor Connector, J2 ELCON CAN DEBUG, J3 ELCON CAN, J4 Conn_02x06_Counter_Clockwise, J5 CAR CAN IN, J6 CAR CAN OUT, J7 BPS CAN DEBUG, J8 BPS CAN, J9 High Side Conn, Q1 SQ2315CES-T1_GE3, Q10 SI7997DP-T1-GE3, Q11 SI7997DP-T1-GE3, Q12 IRLML0030, Q13 PSMN012-100YS, Q14 PSMN012-100YS, Q2 SQ2315CES-T1_GE3, Q3 SQ2315CES-T1_GE3, Q4 IRLML0030, Q5 IRLML0030, Q6 IRLML0030, Q7 IRLML0030, Q8 IRLML0030, Q9 IRLML0030, SW1 SW_SPDT, SW2 BOOT Switch, SW3 RESET Button, T1 HMU1228NL, T2 HMU1228NL, U1 STM32G473VETx, U10 MCP1826S, U11 TPS2117DRLR, U12 LMR51635XDDCR, U13 PESD5V0L2BT, U14 PESD5V0L2BT, U15 TPS2117DRLR, U16 MCP1826S, U17 TPS2121RUXR, U18 CDSOT23-T24CAN, U2 CDSOT23-T24CAN, U3 CDSOT23-T24CAN, U4 ESP32-C6-MINI-1, U5 DRV110APWR, U6 TPS2121RUXR, U7 DRV110APWR, U8 DRV110APWR, U9 EMC2305-1-AP-TR, Y1 Crystal

Commit message: workday
Parts:
- removed the J5 at (147.9, 132.1)
- removed the J6 at (161.3, 132.1)
- removed the J8 at (128.1, 122.0)
- removed the R2 at (150.5, 128.3)
- added D23: VSSAF522-M3/H, LHRS_Passives:SODFL5226X100N, F.Cu at (-74.1, -13.9)
- added D24: VSSAF522-M3/H, LHRS_Passives:SODFL5226X100N, F.Cu at (-74.1, -9.82)
- added FAN2: Conn_01x04, LHRS_Connectors:Molex_Nano-Fit_105309-xx04_1x04_P2.50mm_Vertical, F.Cu at (-78.3, 3.48)
- added FAN4: Conn_01x04, LHRS_Connectors:Molex_Nano-Fit_105309-xx04_1x04_P2.50mm_Vertical, F.Cu at (-69.9, 3.48)
- added R83: 10k, Resistor_SMD:R_0603_1608Metric_Pad0.98x0.95mm_HandSolder, F.Cu at (-81.5, 13.4)
- added R86: 10k, Resistor_SMD:R_0603_1608Metric_Pad0.98x0.95mm_HandSolder, F.Cu at (-81.5, 15.9)
- C56: moved to F.Cu
- J3: value ELCON CAN -> Conn_02x07_Counter_Clockwise; footprint LHRS_Connectors:Molex_Nano-Fit_105309-xx05_1x05_P2.50mm_Vertical -> LHRS_Connectors:Molex_Microfit3.0_02x07_14-Pin-Horizontal-PCB-Receptacle_447641401
- J4: value Conn_02x06_Counter_Clockwise -> CAR CAN DEBUG; footprint Connector_Molex:Molex_Nano-Fit_105310-xx12_2x06_P2.50mm_Vertical -> LHRS_Connectors:Molex_Nano-Fit_105309-xx04_1x04_P2.50mm_Vertical
- moved D22 244.0 mm to (-88.3, -11.3)
- moved FAN1 244.0 mm to (-96.3, -15.3)
- moved FAN3 244.0 mm to (-110.0, -1.10)
- moved C47 238.9 mm to (-94.8, -1.30)
- moved C48 238.9 mm to (-94.8, 0.30)
- moved D21 238.9 mm to (-99.9, -0.49)
- moved R82 238.9 mm to (-99.1, 0.71)
- moved R84 238.9 mm to (-97.3, -0.28)
- moved R85 238.9 mm to (-99.1, 4.19)
- moved R87 238.9 mm to (-91.6, 3.50)
- moved R88 238.9 mm to (-89.9, 3.50)
- moved R89 238.9 mm to (-96.2, 5.48)
- moved U9 238.9 mm to (-95.5, 2.99)
- moved C92 225.4 mm to (372.5, 202.0)
- moved C93 225.4 mm to (370.6, 202.0)
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- renumbered D23 to D25, D24 to D26, D25 to D27, D26 to D28, D27 to D29, D28 to D30, D29 to D31, D30 to D32, FAN2 to FAN3, J13 to J10, J14 to J11, J15 to J12, J16 to J13, J17 to J14, J7 to J5, J9 to J6, J10 to J7, J11 to J8, J12 to J9, R3 to R2, R4 to R3, R91 to R4, R83 to R84, R84 to R85, R85 to R87, R86 to R88, R87 to R89, R88 to R90, R89 to R91, R90 to R92, TP11 to TP10, TP12 to TP11, TP13 to TP12, TP14 to TP13, TP15 to TP14, TP16 to TP15, TP17 to TP16, TP18 to TP17, TP19 to TP18, TP20 to TP19, TP3 to TP2, TP4 to TP3, TP5 to TP4, TP6 to TP5, TP7 to TP6, TP8 to TP7, TP9 to TP8, TP10 to TP9
Connections:
- J3 pad 1: /ELCON_LV+ -> /LVC_LV+
- J3 pad 2: /CHARGER_CAN_H -> /CAR_CAN_H
- J3 pad 3: /CHARGER_CAN_L -> /CAR_CAN_L
- J3 pad 4: GND -> /CAR_SHIELD
- J3 pad 5: Net-(J3-SHIELD) -> /ELCON_LV+
- J4 pad 1: /PDU_LV+ -> +12V
- J4 pad 2: unconnected-(J4-Pin_2-Pad2) -> /CAR_CAN_H
- J4 pad 3: unconnected-(J4-Pin_3-Pad3) -> /CAR_CAN_L
- J4 pad 4: unconnected-(J4-Pin_4-Pad4) -> GND
- R1 pad 1: Net-(J3-SHIELD) -> GND
- R1 pad 2: GND -> /CAR_SHIELD
- U9 pad 10: unconnected-(U9-TACH3-Pad10) -> /Fan/FAN_3_TACH
- U9 pad 13: unconnected-(U9-PWM4-Pad13) -> /Fan/FAN_4_PWM
- U9 pad 14: unconnected-(U9-TACH4-Pad14) -> /Fan/FAN_4_TACH
- U9 pad 9: unconnected-(U9-PWM3-Pad9) -> /Fan/FAN_3_PWM
Routing:
- net GND: track 137.3 -> 5.01 mm, vias 217 -> 3
- net /ESTOP_OUT: track 114.8 -> 0.00 mm, vias 1 -> 0
- net /MOTOR_SENSE: track 106.1 -> 0.00 mm, vias 1 -> 0
- net +3.3V: track 103.6 -> 0.00 mm, vias 36 -> 0
- net /MOTOR_ECON: track 89.8 -> 0.00 mm, vias 2 -> 0
- net /Power/PD_5V_OUT: track 89.0 -> 0.00 mm, vias 4 -> 0
- net /MOTOR_CTRL: track 85.4 -> 0.00 mm, vias 2 -> 0
- net /HV+_SENSE: track 84.3 -> 0.00 mm, vias 3 -> 0
- net /CAR_CAN_L: track 83.4 -> 0.00 mm
- net /FAN_ALERT: track 82.9 -> 0.00 mm, vias 3 -> 0
- net /FAN_SCL: track 82.8 -> 0.00 mm, vias 3 -> 0
- net /FAN_SDA: track 81.3 -> 0.00 mm, vias 3 -> 0
- net /CAR_CAN_H: track 77.9 -> 0.00 mm
- net /BPS_CAN_H: track 72.0 -> 0.00 mm, vias 2 -> 0
- net /HV-_SENSE: track 71.4 -> 0.00 mm, vias 2 -> 0
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