File: hardware/12V_Buck_Boost.kicad_sch (KiCad schematic)
At the start: 20 parts, among them IC7 TPS552872RYQR

Commit message: part numbers
Parts:
- C100, C107, C96, C99: LCSC (none) -> -- mixed values --; LCSC P/N (none) -> C14663; Mouser Part Number (none) -> -- mixed values --; P/N (none) -> MLASH168SB7104KTNA01
- C101, C102, C103, C105, C97: LCSC P/N (none) -> C5448976; P/N (none) -> GGM31CD70J226KE02L
- C104: LCSC P/N (none) -> C105622; P/N (none) -> CL10C470JB8NNNC
- C106: LCSC P/N (none) -> C282075; P/N (none) -> 0603N910J500CT
- C98: LCSC P/N (none) -> C105911; P/N (none) -> -- mixed values --
- IC7: LCSC P/N (none) -> C22427496; P/N (none) -> TPS552872RYQR
- L2: P/N (none) -> 74439369082
- R137: LCSC P/N (none) -> C4117233; P/N (none) -> CR0603-FX-4992ELF
- R139: LCSC P/N (none) -> C22841; P/N (none) -> CR0603-FX-1431ELF
- R140: LCSC P/N (none) -> C7467372; P/N (none) -> ERJ-8CWJR013V
- R141: LCSC P/N (none) -> C25803; P/N (none) -> CRCW0603100KFKEE
- R142: LCSC P/N (none) -> C1854558; P/N (none) -> RNCF0603BTE11K1
