File: hardware/BMS.kicad_sch (KiCad schematic)
At the start: 26 parts, among them IC4 BQ79600PWRQ1, T1 HMU1228NL, T2 HMU1228NL, U13 PESD5V0L2BT, U14 PESD5V0L2BT

Commit message: part numbers
Parts:
- C68, C71: LCSC (none) -> -- mixed values --; LCSC P/N (none) -> C14663; Mouser Part Number (none) -> -- mixed values --; P/N (none) -> MLASH168SB7104KTNA01
- C69, C70: LCSC P/N (none) -> C107083; P/N (none) -> CC0603KRX7R9BB224
- C72, C73, C74, C75, C76, C77: LCSC P/N (none) -> C14665; P/N (none) -> KGM15AR71C101KT
- IC4: LCSC P/N (none) -> C2869947; P/N (none) -> BQ79600PWRQ1
- R108, R109: LCSC (none) -> -- mixed values --; LCSC P/N (none) -> C25804; Manufactuerer (none) -> -- mixed values --; P/N (none) -> CR0603-FX-1002ELF
- R110, R111: LCSC P/N (none) -> C25803; P/N (none) -> CRCW0603100KFKEE
- R112: LCSC P/N (none) -> C22859; P/N (none) -> CRCW060310R0FKEA
- R113, R114: LCSC (none) -> -- mixed values --; LCSC P/N (none) -> C21190; Manufactuerer (none) -> -- mixed values --; P/N (none) -> CRCW06031K00FKEI
- R115, R116, R117, R118: LCSC P/N (none) -> C2907050; P/N (none) -> CR0603-JW-510ELF
- U13, U14: LCSC P/N (none) -> C12324; P/N (none) -> PESD5V0L2BT
