File: hardware/Peripherals.kicad_sch (KiCad schematic)
At the start: 2 parts

Commit message: part numbers
Parts:
- R10: LCSC (none) -> -- mixed values --; LCSC P/N (none) -> C25804; Manufactuerer (none) -> -- mixed values --; P/N CRCW060310K0FKEI -> CR0603-FX-1002ELF
- R9: LCSC P/N (none) -> C2907001; P/N (none) -> AC0603FR-0718KL
Changed lines of the file:
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@@
 			)
 		)
-		(property "P/N" ""
+		(property "P/N" "AC0603FR-0718KL "
 			(at 21.59 114.3 90)
+			(hide yes)
+			(show_name no)
+			(do_not_autoplace no)
+			(effects
+				(font
+					(size 1.27 1.27)
+				)
+			)
+		)
+		(property "LCSC P/N" "C2907001 "
+			(at 21.59 114.3 0)
 			(hide yes)
 			(show_name no)
@@
 			)
 		)
-		(property "Description" "Resistor"
+		(property "Description" "-- mixed values --"
 			(at 21.59 121.92 0)
 			(hide yes)
@@
 			)
 		)
-		(property "P/N" "CRCW060310K0FKEI "
+		(property "P/N" "CR0603-FX-1002ELF "
 			(at 21.59 121.92 90)
 			(hide yes)
 			(show_name no)
+			(do_not_autoplace no)
+			(effects
+				(font
+					(size 1.27 1.27)
+				)
+			)
+		)
+		(property "LCSC" "-- mixed values --"
+			(at 21.59 121.92 0)
+			(hide yes)
+			(show_name no)
+			(do_not_autoplace no)
+			(effects
+				(font
+					(size 1.27 1.27)
+				)
+			)
+		)
+		(property "LCSC P/N" "C25804 "
+			(at 21.59 121.92 0)
+			(hide yes)
+			(show_name no)
+			(do_not_autoplace no)
+			(effects
+				(font
+					(size 1.27 1.27)
+				)
+			)
+		)
+		(property "Manufactuerer" "-- mixed values --"
+			(at 21.59 121.92 0)
+			(hide yes)
+			(show_name no)
