File: hardware/Power_5VMux.kicad_sch (KiCad schematic)
At the start: 6 parts, among them U15 TPS2117DRLR

Commit message: part numbers
Parts:
- C85, C86, C87, C88: LCSC P/N (none) -> C14663; Mfg MLASH168SB7104KTNA01 -> -- mixed values --
- R125: LCSC (none) -> -- mixed values --; LCSC P/N (none) -> C25804; Manufactuerer (none) -> -- mixed values --; P/N CRCW060310K0FKEI -> CR0603-FX-1002ELF
- U15: LCSC P/N (none) -> C22399676
Changed lines of the file:
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@@
 			)
 		)
-		(property "Mfg" "MLASH168SB7104KTNA01"
+		(property "Mfg" "-- mixed values --"
+			(at 88.9 58.42 0)
+			(hide yes)
+			(show_name no)
+			(do_not_autoplace no)
+			(effects
+				(font
+					(size 1.27 1.27)
+				)
+			)
+		)
+		(property "LCSC P/N" "C14663"
 			(at 88.9 58.42 0)
 			(hide yes)
@@
 			)
 		)
-		(property "Mfg" "MLASH168SB7104KTNA01"
+		(property "Mfg" "-- mixed values --"
+			(at 35.56 45.72 0)
+			(hide yes)
+			(show_name no)
+			(do_not_autoplace no)
+			(effects
+				(font
+					(size 1.27 1.27)
+				)
+			)
+		)
+		(property "LCSC P/N" "C14663"
 			(at 35.56 45.72 0)
 			(hide yes)
@@
 			)
 		)
-		(property "Mfg" "MLASH168SB7104KTNA01"
+		(property "Mfg" "-- mixed values --"
+			(at 21.59 45.72 0)
+			(hide yes)
+			(show_name no)
+			(do_not_autoplace no)
+			(effects
+				(font
+					(size 1.27 1.27)
+				)
+			)
+		)
+		(property "LCSC P/N" "C14663"
 			(at 21.59 45.72 0)
 			(hide yes)
@@
 			)
 		)
-		(property "Mfg" "MLASH168SB7104KTNA01"
+		(property "Mfg" "-- mixed values --"
+			(at 39.37 68.58 0)
+			(hide yes)
+			(show_name no)
+			(do_not_autoplace no)
+			(effects
+				(font
+					(size 1.27 1.27)
+				)
+			)
+		)
+		(property "LCSC P/N" "C14663"
 			(at 39.37 68.58 0)
 			(hide yes)
@@
 			)
 		)
+		(property "LCSC P/N" "C22399676 "
+			(at 60.96 62.23 0)
+			(hide yes)
+			(show_name no)
+			(do_not_autoplace no)
+			(effects
+				(font
+					(size 1.27 1.27)
+				)
+			)
+		)
 		(pin "6"
 		)
@@
 			)
 		)
-		(property "Description" "Resistor"
+		(property "Description" "-- mixed values --"
 			(at 76.2 68.58 0)
 			(hide yes)
@@
 			)
 		)
-		(property "P/N" "CRCW060310K0FKEI "
+		(property "P/N" "CR0603-FX-1002ELF "
 			(at 76.2 68.58 90)
 			(hide yes)
 			(show_name no)
+			(do_not_autoplace no)
+			(effects
+				(font
+					(size 1.27 1.27)
+				)
+			)
+		)
+		(property "LCSC" "-- mixed values --"
+			(at 76.2 68.58 0)
+			(hide yes)
+			(show_name no)
+			(do_not_autoplace no)
+			(effects
+				(font
+					(size 1.27 1.27)
+				)
+			)
+		)
+		(property "LCSC P/N" "C25804 "
+			(at 76.2 68.58 0)
+			(hide yes)
+			(show_name no)
+			(do_not_autoplace no)
+			(effects
+				(font
+					(size 1.27 1.27)
+				)
+			)
+		)
+		(property "Manufactuerer" "-- mixed values --"
+			(at 76.2 68.58 0)
+			(hide yes)
+			(show_name no)
