File: hardware/Power_Mux_12V.kicad_sch (KiCad schematic)
At the start: 11 parts, among them U6 TPS2121RUXR

Commit message: part numbers
Parts:
- C34: LCSC (none) -> -- mixed values --; LCSC P/N (none) -> C15849; Manufactuerer (none) -> -- mixed values --; Mouser Part Number (none) -> -- mixed values --; P/N (none) -> CC0603KRX7R9BB105
- R53: LCSC P/N (none) -> C2933240; P/N (none) -> CR0603-FX-5762ELF
- R54, R56, R58, R60: LCSC P/N (none) -> C862232; P/N (none) -> RT0603BRE075KL
- R55: LCSC P/N (none) -> C861518; P/N (none) -> RT0603BRD0767K3L
- R57: LCSC P/N (none) -> C321818; P/N (none) -> CR0603-FX-2612ELF
- R59: LCSC P/N (none) -> C23033; P/N (none) -> RC0603FR-0737K4L
- R61: LCSC P/N (none) -> C2960862; P/N (none) -> RT0603FRE0722K1L
- U6: P/N (none) -> TPS2121RUXR
