File: hardware/Power_Mux_PD.kicad_sch (KiCad schematic)
At the start: 11 parts, among them U17 TPS2121RUXR

Commit message: part numbers
Parts:
- C91: LCSC (none) -> -- mixed values --; LCSC P/N (none) -> C15849; Manufactuerer (none) -> -- mixed values --; Mouser Part Number (none) -> -- mixed values --; P/N (none) -> CC0603KRX7R9BB105
- R126, R132: LCSC P/N (none) -> C2933240; P/N (none) -> CR0603-FX-5762ELF
- R127, R129, R131, R133: LCSC P/N (none) -> C862232; P/N (none) -> RT0603BRE075KL
- R128: LCSC P/N (none) -> C25803; P/N (none) -> CRCW0603100KFKEE
- R130: LCSC P/N (none) -> C321818; P/N (none) -> CR0603-FX-2612ELF
- R134: LCSC P/N (none) -> C2960862; P/N (none) -> RT0603FRE0722K1L
- U17: P/N (none) -> TPS2121RUXR
