File: hardware/100PinMCU.kicad_sch (KiCad schematic)
At the start: 33 parts, among them J11 SWD_Header, J12 SWD, SW1 SW_SPDT, U1 STM32G473VETx, Y1 Crystal

Commit message: part numbers
Parts:
- C10, C12: Mouser Part Number MLASH168SB7104KTNA01 -> -- mixed values --
- C11, C13, C14, C15, C5, C6, C7, C8, C9: LCSC (none) -> -- mixed values --; Mouser Part Number MLASH168SB7104KTNA01 -> -- mixed values --
- C4: Mouser P/N (none) -> -- mixed values --; Mouser Part Number 08055D475KAT4A -> -- mixed values --; P/N GRM21BR61H106KE43K -> GRM21BR61H106KE43L
- J12: now left out of the parts list
- R11, R17: Mouser Part Number CRCW060310K0FKEI -> -- mixed values --; P/N CRCW060310K0FKEI -> CR0603-FX-1002ELF
- SW1: LCSC P/N - -> (none)
Changed lines of the file:
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@@
 			)
 		)
-		(property "Mouser Part Number" "MLASH168SB7104KTNA01"
+		(property "Mouser Part Number" "-- mixed values --"
 			(at 209.55 52.705 0)
 			(hide yes)
@@
 			)
 		)
-		(property "Datasheet" ""
+		(property "Datasheet" "-- mixed values --"
 			(at 196.85 88.265 0)
 			(hide yes)
@@
 			)
 		)
-		(property "Description" "Resistor, US symbol"
+		(property "Description" "-- mixed values --"
 			(at 196.85 88.265 0)
 			(hide yes)
@@
 			)
 		)
-		(property "Mouser Part Number" "CRCW060310K0FKEI "
+		(property "Mouser Part Number" "-- mixed values --"
 			(at 196.85 88.265 0)
 			(hide yes)
@@
 			)
 		)
-		(property "P/N" "CRCW060310K0FKEI "
+		(property "P/N" "CR0603-FX-1002ELF "
 			(at 196.85 88.265 0)
 			(hide yes)
@@
 			)
 		)
-		(property "Description" "Unpolarized capacitor"
+		(property "Description" "-- mixed values --"
 			(at 196.85 99.695 0)
 			(hide yes)
@@
 			)
 		)
-		(property "Mouser Part Number" "MLASH168SB7104KTNA01"
+		(property "Mouser Part Number" "-- mixed values --"
 			(at 196.85 99.695 0)
 			(hide yes)
@@
 			)
 		)
+		(property "LCSC" "-- mixed values --"
+			(at 196.85 99.695 0)
+			(hide yes)
+			(show_name no)
+			(do_not_autoplace no)
+			(effects
+				(font
+					(size 1.27 1.27)
+				)
+			)
+		)
 		(pin "1"
 		)
@@
 			)
 		)
-		(property "Datasheet" ""
+		(property "Datasheet" "-- mixed values --"
 			(at 274.574 104.775 0)
 			(hide yes)
@@
 			)
 		)
-		(property "Description" "Resistor"
+		(property "Description" "-- mixed values --"
 			(at 274.574 104.775 0)
 			(hide yes)
@@
 			)
 		)
-		(property "Datasheet" ""
+		(property "Datasheet" "-- mixed values --"
 			(at 263.144 97.155 0)
 			(hide yes)
@@
 			)
 		)
-		(property "Description" "Resistor"
+		(property "Description" "-- mixed values --"
 			(at 263.144 97.155 0)
 			(hide yes)
@@
 			)
 		)
-		(property "Mouser Part Number" "CRCW060310K0FKEI "
+		(property "Mouser Part Number" "-- mixed values --"
 			(at 263.144 97.155 0)
 			(hide yes)
@@
 			)
 		)
-		(property "P/N" "CRCW060310K0FKEI "
+		(property "P/N" "CR0603-FX-1002ELF "
 			(at 263.144 97.155 0)
 			(hide yes)
@@
 			)
 		)
-		(property "Description" "Unpolarized capacitor"
+		(property "Description" "-- mixed values --"
 			(at 194.31 52.705 0)
 			(hide yes)
@@
 			)
 		)
-		(property "Mouser Part Number" "MLASH168SB7104KTNA01"
+		(property "Mouser Part Number" "-- mixed values --"
 			(at 194.31 52.705 0)
 			(hide yes)
@@
 			)
 		)
+		(property "LCSC" "-- mixed values --"
+			(at 194.31 52.705 0)
+			(hide yes)
+			(show_name no)
+			(do_not_autoplace no)
+			(effects
+				(font
+					(size 1.27 1.27)
+				)
+			)
+		)
 		(pin "1"
 		)
@@
 			)
 		)
-		(property "Description" "Unpolarized capacitor"
+		(property "Description" "-- mixed values --"
 			(at 189.23 27.305 0)
 			(hide yes)
@@
 			)
 		)
-		(property "Mouser Part Number" "MLASH168SB7104KTNA01"
+		(property "Mouser Part Number" "-- mixed values --"
 			(at 189.23 27.305 0)
 			(hide yes)
@@
 			)
 		)
+		(property "LCSC" "-- mixed values --"
+			(at 189.23 27.305 0)
+			(hide yes)
+			(show_name no)
+			(do_not_autoplace no)
+			(effects
+				(font
+					(size 1.27 1.27)
+				)
+			)
+		)
 		(pin "1"
 		)
@@
 			)
 		)
-		(property "Description" "Unpolarized capacitor"
+		(property "Description" "-- mixed values --"
 			(at 214.63 27.305 0)
 			(hide yes)
@@
 			)
 		)
-		(property "Mouser Part Number" "MLASH168SB7104KTNA01"
+		(property "Mouser Part Number" "-- mixed values --"
 			(at 214.63 27.305 0)
 			(hide yes)
@@
 			)
 		)
+		(property "LCSC" "-- mixed values --"
+			(at 214.63 27.305 0)
+			(hide yes)
+			(show_name no)
+			(do_not_autoplace no)
+			(effects
+				(font
+					(size 1.27 1.27)
+				)
+			)
+		)
 		(pin "1"
 		)
@@
 			)
 		)
-		(property "Description" "Unpolarized capacitor"
+		(property "Description" "-- mixed values --"
 			(at 227.33 27.305 0)
 			(hide yes)
@@
 			)
 		)
-		(property "Mouser Part Number" "MLASH168SB7104KTNA01"
+		(property "Mouser Part Number" "-- mixed values --"
 			(at 227.33 27.305 0)
 			(hide yes)
@@
 			)
 		)
+		(property "LCSC" "-- mixed values --"
+			(at 227.33 27.305 0)
+			(hide yes)
+			(show_name no)
+			(do_not_autoplace no)
+			(effects
+				(font
+					(size 1.27 1.27)
+				)
+			)
+		)
 		(pin "1"
 		)
@@
 			)
 		)
-		(property "LCSC P/N" "-"
+		(property "LCSC P/N" ""
 			(at 245.364 92.075 0)
 			(hide yes)
@@
 			)
 		)
-		(property "Description" "Unpolarized capacitor"
+		(property "Description" "-- mixed values --"
 			(at 179.07 27.305 0)
 			(hide yes)
@@
 			)
 		)
-		(property "Mouser Part Number" "08055D475KAT4A"
+		(property "Mouser Part Number" "-- mixed values --"
 			(at 179.07 27.305 0)
 			(hide yes)
@@
 			)
 		)
-		(property "P/N" "GRM21BR61H106KE43K"
+		(property "P/N" "GRM21BR61H106KE43L "
 			(at 179.07 27.305 0)
 			(hide yes)
@@
 			)
 		)
+		(property "Mouser P/N" "-- mixed values --"
+			(at 179.07 27.305 0)
+			(hide yes)
+			(show_name no)
+			(do_not_autoplace no)
+			(effects
+				(font
+					(size 1.27 1.27)
+				)
+			)
+		)
 		(pin "1"
 		)
@@
 			)
 		)
-		(property "Description" "Unpolarized capacitor"
+		(property "Description" "-- mixed values --"
 			(at 179.07 52.705 0)
 			(hide yes)
@@
 			)
 		)
-		(property "Mouser Part Number" "MLASH168SB7104KTNA01"
+		(property "Mouser Part Number" "-- mixed values --"
 			(at 179.07 52.705 0)
 			(hide yes)
@@
 			)
 		)
+		(property "LCSC" "-- mixed values --"
+			(at 179.07 52.705 0)
+			(hide yes)
+			(show_name no)
+			(do_not_autoplace no)
+			(effects
+				(font
+					(size 1.27 1.27)
+				)
+			)
+		)
 		(pin "1"
 		)
@@
 			)
 		)
-		(property "Mouser Part Number" "MLASH168SB7104KTNA01"
+		(property "Mouser Part Number" "-- mixed values --"
 			(at 224.79 52.705 0)
 			(hide yes)
@@
 			)
 		)
-		(property "Datasheet" ""
+		(property "Datasheet" "-- mixed values --"
 			(at 255.27 150.495 0)
 			(hide yes)
@@
 			)
 		)
-		(property "Description" "Resistor"
+		(property "Description" "-- mixed values --"
 			(at 255.27 150.495 0)
 			(hide yes)
@@
 			)
 		)
-		(property "Description" "Unpolarized capacitor"
+		(property "Description" "-- mixed values --"
 			(at 262.89 56.515 0)
 			(hide yes)
@@
 			)
 		)
-		(property "Mouser Part Number" "MLASH168SB7104KTNA01"
+		(property "Mouser Part Number" "-- mixed values --"
 			(at 262.89 56.515 0)
 			(hide yes)
@@
 			)
 		)
+		(property "LCSC" "-- mixed values --"
+			(at 262.89 56.515 0)
+			(hide yes)
+			(show_name no)
+			(do_not_autoplace no)
+			(effects
+				(font
+					(size 1.27 1.27)
+				)
+			)
+		)
 		(pin "1"
 		)
@@
 			)
 		)
-		(property "Description" "Unpolarized capacitor"
+		(property "Description" "-- mixed values --"
 			(at 201.93 27.305 0)
 			(hide yes)
@@
 			)
 		)
-		(property "Mouser Part Number" "MLASH168SB7104KTNA01"
+		(property "Mouser Part Number" "-- mixed values --"
 			(at 201.93 27.305 0)
 			(hide yes)
@@
 			)
 		)
+		(property "LCSC" "-- mixed values --"
+			(at 201.93 27.305 0)
+			(hide yes)
+			(show_name no)
+			(do_not_autoplace no)
+			(effects
+				(font
+					(size 1.27 1.27)
+				)
+			)
+		)
 		(pin "1"
 		)
@@
 			)
 		)
-		(property "Datasheet" ""
+		(property "Datasheet" "-- mixed values --"
 			(at 247.65 150.495 0)
 			(hide yes)
@@
 			)
 		)
-		(property "Description" "Resistor"
+		(property "Description" "-- mixed values --"
 			(at 247.65 150.495 0)
 			(hide yes)
@@
 			)
 		)
-		(property "Datasheet" ""
+		(property "Datasheet" "-- mixed values --"
 			(at 262.89 150.495 0)
 			(hide yes)
@@
 			)
 		)
-		(property "Description" "Resistor"
+		(property "Description" "-- mixed values --"
 			(at 262.89 150.495 0)
 			(hide yes)
@@
 			)
 		)
-		(property "Description" "Unpolarized capacitor"
+		(property "Description" "-- mixed values --"
 			(at 240.03 27.305 0)
 			(hide yes)
@@
 			)
 		)
-		(property "Mouser Part Number" "MLASH168SB7104KTNA01"
+		(property "Mouser Part Number" "-- mixed values --"
 			(at 240.03 27.305 0)
 			(hide yes)
@@
 			)
 		)
+		(property "LCSC" "-- mixed values --"
+			(at 240.03 27.305 0)
+			(hide yes)
+			(show_name no)
+			(do_not_autoplace no)
+			(effects
+				(font
+					(size 1.27 1.27)
+				)
+			)
+		)
 		(pin "1"
 		)
@@
 		(body_style 1)
 		(exclude_from_sim no)
-		(in_bom yes)
+		(in_bom no)
 		(on_board yes)
 		(in_pos_files yes)

Commit message: workday
Parts:
- renumbered J11 to J8, J12 to J9
Changed lines of the file:
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@@
 		(in_pos_files yes)
 		(dnp no)
-		(property "Reference" "J11"
+		(property "Reference" "J8"
 			(at 225.552 127.889 0)
 			(show_name no)
@@
 			(project "PS-BPSLeader"
 				(path "/d4a4ed4f-0983-4aef-b212-0e3284ab3963/5da56964-fa04-4fec-bdfe-c6acfeda5c9a/972ee48b-c33c-4022-a95a-ebc71c386daa"
-					(reference "J11")
+					(reference "J8")
 					(unit 1)
 				)
@@
 		(in_pos_files yes)
 		(dnp no)
-		(property "Reference" "J12"
+		(property "Reference" "J9"
 			(at 224.536 145.669 0)
 			(show_name no)
@@
 			(project "PS-BPSLeader"
 				(path "/d4a4ed4f-0983-4aef-b212-0e3284ab3963/5da56964-fa04-4fec-bdfe-c6acfeda5c9a/972ee48b-c33c-4022-a95a-ebc71c386daa"
-					(reference "J12")
+					(reference "J9")
 					(unit 1)
 				)
