File: hardware/12VBuck.kicad_sch (KiCad schematic)
At the start: 12 parts, among them U12 LMR51635XDDCR

Commit message: reviewed
Parts:
- TP11, TP12, TP14: now not fitted; now left out of the parts list
- TP13: now not fitted

Commit message: part numbers
Parts:
- C55: LCSC P/N C6962403 -> C105911; P/N 08055D475KAT4A -> -- mixed values --
Changed lines of the file:
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@@
 			)
 		)
-		(property "Description" "Unpolarized capacitor, small symbol"
+		(property "Description" "-- mixed values --"
 			(at 96.5669 58.5802 0)
 			(hide yes)
@@
 			)
 		)
-		(property "LCSC P/N" "C6962403"
+		(property "LCSC P/N" "C105911 "
 			(at 96.5669 58.5802 0)
 			(hide yes)
@@
 			)
 		)
-		(property "P/N" "08055D475KAT4A"
+		(property "P/N" "-- mixed values --"
 			(at 96.5669 58.5802 0)
 			(hide yes)

Commit message: workday
Parts:
- renumbered R89 to R91, R90 to R92, TP11 to TP10, TP12 to TP11, TP13 to TP12, TP14 to TP13
Changed lines of the file:
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@@
 		(dnp no)
 		(fields_autoplaced yes)
-		(property "Reference" "#FLG04"
+		(property "Reference" "#FLG05"
 			(at 152.4469 51.5952 0)
 			(hide yes)
@@
 			(project "PS-BPSLeader"
 				(path "/d4a4ed4f-0983-4aef-b212-0e3284ab3963/69244dac-f10b-499c-a2b2-3cdf1370aa1f/408035a5-5a4d-4c9d-abf0-417376518132"
-					(reference "#FLG04")
+					(reference "#FLG05")
 					(unit 1)
 				)
@@
 		(in_pos_files yes)
 		(dnp yes)
-		(property "Reference" "TP13"
+		(property "Reference" "TP12"
 			(at 245.1569 95.9181 0)
 			(hide yes)
@@
 			(project "PS-BPSLeader"
 				(path "/d4a4ed4f-0983-4aef-b212-0e3284ab3963/69244dac-f10b-499c-a2b2-3cdf1370aa1f/408035a5-5a4d-4c9d-abf0-417376518132"
-					(reference "TP13")
+					(reference "TP12")
 					(unit 1)
 				)
@@
 		(in_pos_files yes)
 		(dnp yes)
-		(property "Reference" "TP12"
+		(property "Reference" "TP11"
 			(at 232.4569 108.6181 0)
 			(hide yes)
@@
 			(project "PS-BPSLeader"
 				(path "/d4a4ed4f-0983-4aef-b212-0e3284ab3963/69244dac-f10b-499c-a2b2-3cdf1370aa1f/408035a5-5a4d-4c9d-abf0-417376518132"
-					(reference "TP12")
+					(reference "TP11")
 					(unit 1)
 				)
@@
 		(in_pos_files yes)
 		(dnp yes)
-		(property "Reference" "TP14"
+		(property "Reference" "TP13"
 			(at 245.1569 108.6181 0)
 			(hide yes)
@@
 			(project "PS-BPSLeader"
 				(path "/d4a4ed4f-0983-4aef-b212-0e3284ab3963/69244dac-f10b-499c-a2b2-3cdf1370aa1f/408035a5-5a4d-4c9d-abf0-417376518132"
-					(reference "TP14")
+					(reference "TP13")
 					(unit 1)
 				)
@@
 		(dnp no)
 		(fields_autoplaced yes)
-		(property "Reference" "#FLG06"
+		(property "Reference" "#FLG07"
 			(at 184.1969 56.6752 0)
 			(hide yes)
@@
 			(project "PS-BPSLeader"
 				(path "/d4a4ed4f-0983-4aef-b212-0e3284ab3963/69244dac-f10b-499c-a2b2-3cdf1370aa1f/408035a5-5a4d-4c9d-abf0-417376518132"
-					(reference "#FLG06")
+					(reference "#FLG07")
 					(unit 1)
 				)
@@
 		(in_pos_files yes)
 		(dnp no)
-		(property "Reference" "#FLG05"
+		(property "Reference" "#FLG06"
 			(at 152.4469 56.6752 0)
 			(hide yes)
@@
 			(project "PS-BPSLeader"
 				(path "/d4a4ed4f-0983-4aef-b212-0e3284ab3963/69244dac-f10b-499c-a2b2-3cdf1370aa1f/408035a5-5a4d-4c9d-abf0-417376518132"
-					(reference "#FLG05")
+					(reference "#FLG06")
 					(unit 1)
 				)
@@
 		(dnp no)
 		(fields_autoplaced yes)
-		(property "Reference" "R89"
+		(property "Reference" "R91"
 			(at 229.9169 57.3101 0)
 			(show_name no)
@@
 			(project "PS-BPSLeader"
 				(path "/d4a4ed4f-0983-4aef-b212-0e3284ab3963/69244dac-f10b-499c-a2b2-3cdf1370aa1f/408035a5-5a4d-4c9d-abf0-417376518132"
-					(reference "R89")
+					(reference "R91")
 					(unit 1)
 				)
@@
 		(in_pos_files yes)
 		(dnp yes)
-		(property "Reference" "TP11"
+		(property "Reference" "TP10"
 			(at 232.4569 95.9181 0)
 			(hide yes)
@@
 			(project "PS-BPSLeader"
 				(path "/d4a4ed4f-0983-4aef-b212-0e3284ab3963/69244dac-f10b-499c-a2b2-3cdf1370aa1f/408035a5-5a4d-4c9d-abf0-417376518132"
-					(reference "TP11")
+					(reference "TP10")
 					(unit 1)
 				)
@@
 		(dnp no)
 		(fields_autoplaced yes)
-		(property "Reference" "R90"
+		(property "Reference" "R92"
 			(at 229.9169 64.9301 0)
 			(show_name no)
@@
 			(project "PS-BPSLeader"
 				(path "/d4a4ed4f-0983-4aef-b212-0e3284ab3963/69244dac-f10b-499c-a2b2-3cdf1370aa1f/408035a5-5a4d-4c9d-abf0-417376518132"
-					(reference "R90")
+					(reference "R92")
 					(unit 1)
 				)
@@
 		(dnp no)
 		(fields_autoplaced yes)
-		(property "Reference" "#FLG03"
+		(property "Reference" "#FLG04"
 			(at 91.4869 51.5952 0)
 			(hide yes)
@@
 			(project "PS-BPSLeader"
 				(path "/d4a4ed4f-0983-4aef-b212-0e3284ab3963/69244dac-f10b-499c-a2b2-3cdf1370aa1f/408035a5-5a4d-4c9d-abf0-417376518132"
-					(reference "#FLG03")
-					(unit 1)
-				)
+					(reference "#FLG04")
+					(unit 1)
+				)
