File: hardware/12VBuck.kicad_sch (KiCad schematic)
At the start: 12 parts, among them U12 LMR51635XDDCR

Commit message: fixed fan chip footprint and buck output capacitors
Parts:
- added C?: 22u, Capacitor_SMD:C_1210_3225Metric_Pad1.33x2.70mm_HandSolder, symbol Device:C_Small
- added C?: 4.7u, Capacitor_SMD:C_1210_3225Metric_Pad1.33x2.70mm_HandSolder, symbol Device:C_Small
- C58: value 47u -> 22u
Connections:
- new net: C?.2, C?.2
