File: hardware/ESP32.kicad_sch (KiCad schematic)
At the start: 21 parts, among them J13 USB_C_Receptacle_USB2.0_16P, SW2 BOOT Switch, SW3 RESET Button, U4 ESP32-C6-MINI-1

Commit message: part numbers
Parts:
- C24, C25, C26, C27, R23, R24: Mfg (none) -> -- mixed values --
- J13: P/N USB4105-GF-A -> -- mixed values --
- R25, R26, R27: Mouser Part Number (none) -> -- mixed values --; P/N CRCW060310K0FKEI -> CR0603-FX-1002ELF
Changed lines of the file:
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@@
 			)
 		)
-		(property "Datasheet" "kicad-embed://dcrcwe3.pdf"
+		(property "Datasheet" "-- mixed values --"
 			(at 200.66 34.29 0)
 			(hide yes)
@@
 			)
 		)
-		(property "Description" "resistor"
+		(property "Description" "-- mixed values --"
 			(at 200.66 34.29 0)
 			(hide yes)
@@
 			)
 		)
-		(property "Datasheet" "kicad-embed://GRM21BR61H106KE43_01A.pdf"
+		(property "Datasheet" "-- mixed values --"
 			(at 71.12 78.74 0)
 			(hide yes)
@@
 		)
 		(property "LCSC P/N" "C440198"
+			(at 71.12 78.74 0)
+			(hide yes)
+			(show_name no)
+			(do_not_autoplace no)
+			(effects
+				(font
+					(size 1.27 1.27)
+				)
+			)
+		)
+		(property "Mfg" "-- mixed values --"
 			(at 71.12 78.74 0)
 			(hide yes)
@@
 			)
 		)
+		(property "Mfg" "-- mixed values --"
+			(at 148.59 74.93 0)
+			(hide yes)
+			(show_name no)
+			(do_not_autoplace no)
+			(effects
+				(font
+					(size 1.27 1.27)
+				)
+			)
+		)
 		(pin "2"
 		)
@@
 			)
 		)
-		(property "Datasheet" "kicad-embed://dcrcwe3.pdf"
+		(property "Datasheet" "-- mixed values --"
 			(at 200.66 39.37 0)
 			(hide yes)
@@
 			)
 		)
-		(property "Description" "resistor"
+		(property "Description" "-- mixed values --"
 			(at 200.66 39.37 0)
 			(hide yes)
@@
 			)
 		)
-		(property "Datasheet" "kicad-embed://GRM21BR61H106KE43_01A.pdf"
+		(property "Datasheet" "-- mixed values --"
 			(at 139.7 74.93 0)
 			(hide yes)
@@
 		)
 		(property "LCSC P/N" "C440198"
+			(at 139.7 74.93 0)
+			(hide yes)
+			(show_name no)
+			(do_not_autoplace no)
+			(effects
+				(font
+					(size 1.27 1.27)
+				)
+			)
+		)
+		(property "Mfg" "-- mixed values --"
 			(at 139.7 74.93 0)
 			(hide yes)
@@
 			)
 		)
-		(property "Datasheet" "kicad-embed://dcrcwe3.pdf"
+		(property "Datasheet" "-- mixed values --"
 			(at 199.39 106.68 0)
 			(hide yes)
@@
 			)
 		)
-		(property "Description" "resistor"
+		(property "Description" "-- mixed values --"
 			(at 199.39 106.68 0)
 			(hide yes)
@@
 			)
 		)
-		(property "P/N" "CRCW060310K0FKEI "
+		(property "P/N" "CR0603-FX-1002ELF "
 			(at 199.39 106.68 90)
 			(hide yes)
@@
 					(size 1.27 1.27)
 					(thickness 0.1588)
+				)
+			)
+		)
+		(property "Mouser Part Number" "-- mixed values --"
+			(at 199.39 106.68 90)
+			(hide yes)
+			(show_name no)
+			(do_not_autoplace no)
+			(effects
+				(font
+					(size 1.27 1.27)
 				)
 			)
@@
 			)
 		)
-		(property "Datasheet" "kicad-embed://dcrcwe3.pdf"
+		(property "Datasheet" "-- mixed values --"
 			(at 107.95 34.29 0)
 			(hide yes)
@@
 			)
 		)
-		(property "Description" "resistor"
+		(property "Description" "-- mixed values --"
 			(at 107.95 34.29 0)
 			(hide yes)
@@
 			)
 		)
-		(property "P/N" "CRCW060310K0FKEI "
+		(property "P/N" "CR0603-FX-1002ELF "
 			(at 107.95 34.29 90)
 			(hide yes)
@@
 					(size 1.27 1.27)
 					(thickness 0.1588)
+				)
+			)
+		)
+		(property "Mouser Part Number" "-- mixed values --"
+			(at 107.95 34.29 90)
+			(hide yes)
+			(show_name no)
+			(do_not_autoplace no)
+			(effects
+				(font
+					(size 1.27 1.27)
 				)
 			)
@@
 			)
 		)
-		(property "Datasheet" "kicad-embed://dcrcwe3.pdf"
+		(property "Datasheet" "-- mixed values --"
 			(at 54.61 80.01 0)
 			(hide yes)
@@
 			)
 		)
-		(property "Description" "Resistor, US symbol"
+		(property "Description" "-- mixed values --"
 			(at 54.61 80.01 0)
 			(hide yes)
@@
 					(size 1.27 1.27)
 					(thickness 0.1588)
+				)
+			)
+		)
+		(property "Mfg" "-- mixed values --"
+			(at 54.61 80.01 90)
+			(hide yes)
+			(show_name no)
+			(do_not_autoplace no)
+			(effects
+				(font
+					(size 1.27 1.27)
 				)
 			)
@@
 			)
 		)
-		(property "Datasheet" "kicad-embed://dcrcwe3.pdf"
+		(property "Datasheet" "-- mixed values --"
 			(at 157.48 27.94 0)
 			(hide yes)
@@
 			)
 		)
-		(property "Description" "resistor"
+		(property "Description" "-- mixed values --"
 			(at 157.48 27.94 0)
 			(hide yes)
@@
 			)
 		)
-		(property "P/N" "CRCW060310K0FKEI "
+		(property "P/N" "CR0603-FX-1002ELF "
 			(at 157.48 27.94 90)
 			(hide yes)
@@
 					(size 1.27 1.27)
 					(thickness 0.1588)
+				)
+			)
+		)
+		(property "Mouser Part Number" "-- mixed values --"
+			(at 157.48 27.94 0)
+			(hide yes)
+			(show_name no)
+			(do_not_autoplace no)
+			(effects
+				(font
+					(size 1.27 1.27)
 				)
 			)
@@
 			)
 		)
+		(property "Mfg" "-- mixed values --"
+			(at 157.48 38.1 0)
+			(hide yes)
+			(show_name no)
+			(do_not_autoplace no)
+			(effects
+				(font
+					(size 1.27 1.27)
+				)
+			)
+		)
 		(pin "2"
 		)
@@
 			)
 		)
-		(property "Datasheet" "kicad-embed://dcrcwe3.pdf"
+		(property "Datasheet" "-- mixed values --"
 			(at 54.61 77.47 0)
 			(hide yes)
@@
 			)
 		)
-		(property "Description" "Resistor, US symbol"
+		(property "Description" "-- mixed values --"
 			(at 54.61 77.47 0)
 			(hide yes)
@@
 					(size 1.27 1.27)
 					(thickness 0.1588)
+				)
+			)
+		)
+		(property "Mfg" "-- mixed values --"
+			(at 54.61 77.47 90)
+			(hide yes)
+			(show_name no)
+			(do_not_autoplace no)
+			(effects
+				(font
+					(size 1.27 1.27)
 				)
 			)
@@
 			)
 		)
-		(property "Datasheet" "kicad-embed://usb4105-spec.pdf"
+		(property "Datasheet" "-- mixed values --"
 			(at 35.56 87.63 0)
 			(hide yes)
@@
 			)
 		)
-		(property "P/N" "USB4105-GF-A"
+		(property "P/N" "-- mixed values --"
 			(at 31.75 87.63 0)
 			(hide yes)
@@
 			)
 		)
-		(property "Datasheet" "kicad-embed://dcrcwe3.pdf"
+		(property "Datasheet" "-- mixed values --"
 			(at 200.66 24.13 0)
 			(hide yes)
@@
 			)
 		)
-		(property "Description" "resistor"
+		(property "Description" "-- mixed values --"
 			(at 200.66 24.13 0)
 			(hide yes)

Commit message: ehehe
Parts:
- J13: P/N -- mixed values -- -> USB4105-GF-A
Changed lines of the file:
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@@
 			)
 		)
-		(property "P/N" "-- mixed values --"
+		(property "P/N" "USB4105-GF-A"
 			(at 31.75 87.63 0)
 			(hide yes)

Commit message: workday
Parts:
- renumbered J13 to J10
Changed lines of the file:
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@@
 		(dnp no)
 		(fields_autoplaced yes)
-		(property "Reference" "J13"
+		(property "Reference" "J10"
 			(at 31.75 64.77 0)
 			(show_name no)
@@
 			(project "PS-BPSLeader"
 				(path "/d4a4ed4f-0983-4aef-b212-0e3284ab3963/5da56964-fa04-4fec-bdfe-c6acfeda5c9a/37240678-40e7-4b21-a99e-c284d3b12e6a"
-					(reference "J13")
+					(reference "J10")
 					(unit 1)
 				)
