File: hardware/ESP32_LDO.kicad_sch (KiCad schematic)
At the start: 5 parts, among them U10 MCP1826S

Commit message: part numbers
Parts:
- C49, C50: Mouser P/N GRM21BR61H106KE43K -> -- mixed values --; Mouser Part Number (none) -> -- mixed values --; P/N (none) -> GRM21BR61H106KE43L
Changed lines of the file:
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@@
 			)
 		)
-		(property "Description" "Unpolarized capacitor, small symbol"
+		(property "Description" "-- mixed values --"
 			(at 165.1 69.85 0)
 			(hide yes)
@@
 			)
 		)
-		(property "Mouser P/N" "GRM21BR61H106KE43K"
+		(property "Mouser P/N" "-- mixed values --"
 			(at 165.1 69.85 0)
 			(hide yes)
@@
 		)
 		(property "LCSC P/N" "C440198"
+			(at 165.1 69.85 0)
+			(hide yes)
+			(show_name no)
+			(do_not_autoplace no)
+			(effects
+				(font
+					(size 1.27 1.27)
+				)
+			)
+		)
+		(property "Mouser Part Number" "-- mixed values --"
+			(at 165.1 69.85 0)
+			(hide yes)
+			(show_name no)
+			(do_not_autoplace no)
+			(effects
+				(font
+					(size 1.27 1.27)
+				)
+			)
+		)
+		(property "P/N" "GRM21BR61H106KE43L "
 			(at 165.1 69.85 0)
 			(hide yes)
@@
 			)
 		)
-		(property "Description" "Unpolarized capacitor, small symbol"
-			(at 139.7 69.85 0)
-			(hide yes)
-			(show_name no)
-			(do_not_autoplace no)
-			(effects
-				(font
-					(size 1.27 1.27)
-				)
-			)
-		)
-		(property "Mouser P/N" "GRM21BR61H106KE43K"
+		(property "Description" "-- mixed values --"
+			(at 139.7 69.85 0)
+			(hide yes)
+			(show_name no)
+			(do_not_autoplace no)
+			(effects
+				(font
+					(size 1.27 1.27)
+				)
+			)
+		)
+		(property "Mouser P/N" "-- mixed values --"
 			(at 139.7 69.85 0)
 			(hide yes)
@@
 			(at 139.7 69.85 0)
 			(hide yes)
+			(show_name no)
+			(do_not_autoplace no)
+			(effects
+				(font
+					(size 1.27 1.27)
+				)
+			)
+		)
+		(property "Mouser Part Number" "-- mixed values --"
+			(at 139.7 69.85 0)
+			(hide yes)
+			(show_name no)
+			(do_not_autoplace no)
+			(effects
+				(font
+					(size 1.27 1.27)
+				)
+			)
+		)
+		(property "P/N" "GRM21BR61H106KE43L "
+			(at 139.7 69.85 0)
+			(hide yes)

Commit message: workday
Parts:
- renumbered D23 to D25
Changed lines of the file:
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@@
 		(dnp no)
 		(fields_autoplaced yes)
-		(property "Reference" "D23"
+		(property "Reference" "D25"
 			(at 133.604 57.15 0)
 			(show_name no)
@@
 			(project "PS-BPSLeader"
 				(path "/d4a4ed4f-0983-4aef-b212-0e3284ab3963/5da56964-fa04-4fec-bdfe-c6acfeda5c9a/92d40a22-22a8-4e19-ae2b-d2176aa2e41e"
-					(reference "D23")
+					(reference "D25")
 					(unit 1)
 				)
