File: hardware/ESP32_Power_Mux.kicad_sch (KiCad schematic)
At the start: 6 parts, among them U11 TPS2117DRLR

Commit message: part numbers
Parts:
- C51, C52, C53, C54: LCSC P/N (none) -> C14663; Mfg MLASH168SB7104KTNA01 -> -- mixed values --
- R88: LCSC (none) -> -- mixed values --; LCSC P/N (none) -> C25804; Manufactuerer (none) -> -- mixed values --; P/N CRCW060310K0FKEI -> CR0603-FX-1002ELF
- U11: LCSC P/N (none) -> C22399676
Changed lines of the file:
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@@
 			)
 		)
-		(property "Mfg" "MLASH168SB7104KTNA01"
+		(property "Mfg" "-- mixed values --"
+			(at 88.9 58.42 0)
+			(hide yes)
+			(show_name no)
+			(do_not_autoplace no)
+			(effects
+				(font
+					(size 1.27 1.27)
+				)
+			)
+		)
+		(property "LCSC P/N" "C14663"
 			(at 88.9 58.42 0)
 			(hide yes)
@@
 			)
 		)
-		(property "Description" "Resistor"
+		(property "Description" "-- mixed values --"
 			(at 76.2 68.58 0)
 			(hide yes)
@@
 			)
 		)
-		(property "P/N" "CRCW060310K0FKEI "
+		(property "P/N" "CR0603-FX-1002ELF "
 			(at 76.2 68.58 90)
+			(hide yes)
+			(show_name no)
+			(do_not_autoplace no)
+			(effects
+				(font
+					(size 1.27 1.27)
+				)
+			)
+		)
+		(property "LCSC" "-- mixed values --"
+			(at 76.2 68.58 0)
+			(hide yes)
+			(show_name no)
+			(do_not_autoplace no)
+			(effects
+				(font
+					(size 1.27 1.27)
+				)
+			)
+		)
+		(property "LCSC P/N" "C25804 "
+			(at 76.2 68.58 0)
+			(hide yes)
+			(show_name no)
+			(do_not_autoplace no)
+			(effects
+				(font
+					(size 1.27 1.27)
+				)
+			)
+		)
+		(property "Manufactuerer" "-- mixed values --"
+			(at 76.2 68.58 0)
 			(hide yes)
 			(show_name no)
@@
 			)
 		)
-		(property "Mfg" "MLASH168SB7104KTNA01"
+		(property "Mfg" "-- mixed values --"
+			(at 21.59 45.72 0)
+			(hide yes)
+			(show_name no)
+			(do_not_autoplace no)
+			(effects
+				(font
+					(size 1.27 1.27)
+				)
+			)
+		)
+		(property "LCSC P/N" "C14663"
 			(at 21.59 45.72 0)
 			(hide yes)
@@
 			)
 		)
+		(property "LCSC P/N" "C22399676 "
+			(at 60.96 62.23 0)
+			(hide yes)
+			(show_name no)
+			(do_not_autoplace no)
+			(effects
+				(font
+					(size 1.27 1.27)
+				)
+			)
+		)
 		(pin "6"
 		)
@@
 			)
 		)
-		(property "Mfg" "MLASH168SB7104KTNA01"
+		(property "Mfg" "-- mixed values --"
+			(at 39.37 68.58 0)
+			(hide yes)
+			(show_name no)
+			(do_not_autoplace no)
+			(effects
+				(font
+					(size 1.27 1.27)
+				)
+			)
+		)
+		(property "LCSC P/N" "C14663"
 			(at 39.37 68.58 0)
 			(hide yes)
@@
 			)
 		)
-		(property "Mfg" "MLASH168SB7104KTNA01"
+		(property "Mfg" "-- mixed values --"
 			(at 35.56 45.72 0)
 			(hide yes)
+			(show_name no)
+			(do_not_autoplace no)
+			(effects
+				(font
+					(size 1.27 1.27)
+				)
+			)
+		)
+		(property "LCSC P/N" "C14663"
+			(at 35.56 45.72 0)
+			(hide yes)

Commit message: workday
Parts:
- renumbered R88 to R90
Changed lines of the file:
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@@
 		(in_pos_files yes)
 		(dnp no)
-		(property "Reference" "R88"
+		(property "Reference" "R90"
 			(at 78.994 67.564 0)
 			(show_name no)
@@
 			(project "PS-BPSLeader"
 				(path "/d4a4ed4f-0983-4aef-b212-0e3284ab3963/5da56964-fa04-4fec-bdfe-c6acfeda5c9a/c396b043-4a62-4d2b-b629-091a6c3457ae"
-					(reference "R88")
+					(reference "R90")
 					(unit 1)
 				)
