File: hardware/ESTOP.kicad_sch (KiCad schematic)
At the start: 22 parts, among them J14 Conn_01x02, Q1 SQ2315CES-T1_GE3, Q2 SQ2315CES-T1_GE3, Q3 SQ2315CES-T1_GE3

Commit message: part numbers
Parts:
- ESTOP1, ESTOP2, ESTOP3: LCSC P/N (none) -> C84263
- Q1, Q2, Q3: LCSC P/N (none) -> C10487; P/N (none) -> SQ2315CES-T1_GE3
- R31, R32, R33, R37, R38, R39: LCSC C25804 -> -- mixed values --; LCSC P/N (none) -> C25804; Manufactuerer Vishay -> -- mixed values --; P/N CRCW060310K0FKEI -> CR0603-FX-1002ELF
- R34, R35, R36: LCSC C23179 -> -- mixed values --; LCSC P/N (none) -> C21190; Manufactuerer Vishay -> -- mixed values --; P/N CRCW0603120RFKEC -> CRCW06031K00FKEI
- R40, R41, R42: LCSC P/N (none) -> C4216; P/N CRCW060310K0FKEI -> CRCW060333K0FKEA

Commit message: workday
Parts:
- renumbered J14 to J11
Changed lines of the file:
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@@
 		(in_pos_files yes)
 		(dnp no)
-		(property "Reference" "J14"
+		(property "Reference" "J11"
 			(at 102.362 84.836 0)
 			(hide yes)
@@
 			(project "PS-BPSLeader"
 				(path "/d4a4ed4f-0983-4aef-b212-0e3284ab3963/ff3d6d8a-5585-4a16-aaa1-d2e71ebe7413"
-					(reference "J14")
+					(reference "J11")
 					(unit 1)
 				)
