File: hardware/Fan.kicad_sch (KiCad schematic)
At the start: 13 parts, among them U9 EMC2305-1-AP-TR

Commit message: workday
Parts:
- added D23, D24: VSSAF522-M3/H, LHRS_Passives:SODFL5226X100N, symbol Diode:C3D25170H
- added FAN2, FAN4: Conn_01x04, LHRS_Connectors:Molex_Nano-Fit_105309-xx04_1x04_P2.50mm_Vertical, symbol Connector_Generic:Conn_01x04
- added R83, R86: 10k, Resistor_SMD:R_0603_1608Metric_Pad0.98x0.95mm_HandSolder, symbol Device:R
- renumbered FAN2 to FAN3, R83 to R84, R84 to R85, R85 to R87, R86 to R88, R87 to R89
Connections:
- net 12V: now also D23.1 (K), D24.1 (K), FAN2.1 (Pin_1), FAN4.1 (Pin_1)
- net 3V3: now also R83.1, R86.1
- net GND: now also D23.2 (A), D24.2 (A), FAN2.4 (Pin_4), FAN4.4 (Pin_4)
- net FAN_3_TACH: now reaches U9.10 (TACH3)
- net FAN_3_TACH: now also FAN2.2 (Pin_2), R83.2
- net FAN_4_PWM: now reaches U9.13 (PWM4)
- net FAN_4_PWM: now also FAN4.3 (Pin_3)
- net FAN_4_TACH: now reaches U9.14 (TACH4)
- net FAN_4_TACH: now also FAN4.2 (Pin_2), R86.2
- net FAN_3_PWM: now reaches U9.9 (PWM3)
- net FAN_3_PWM: now also FAN2.3 (Pin_3)
- no-connect marks 6 -> 2
Other:
- note removed: "Fan Controller"
- note removed: "How many fans?"
- moved on the sheet: D21, D22
