File: hardware/Fan.kicad_sch (KiCad schematic)
At the start: 13 parts, among them U9 EMC2305-1-AP-TR

Commit message: reviewed
Parts:
- FAN1, FAN2: footprint Connector_Molex:Molex_Nano-Fit_105309-xx04_1x04_P2.50mm_Vertical -> LHRS_Connectors:Molex_Nano-Fit_105309-xx04_1x04_P2.50mm_Vertical
Changed lines of the file:
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@@
 			)
 		)
-		(property "Footprint" "Connector_Molex:Molex_Nano-Fit_105309-xx04_1x04_P2.50mm_Vertical"
+		(property "Footprint" "LHRS_Connectors:Molex_Nano-Fit_105309-xx04_1x04_P2.50mm_Vertical"
 			(at 85.09 101.6 0)
 			(hide yes)
@@
 			)
 		)
-		(property "Footprint" "Connector_Molex:Molex_Nano-Fit_105309-xx04_1x04_P2.50mm_Vertical"
+		(property "Footprint" "LHRS_Connectors:Molex_Nano-Fit_105309-xx04_1x04_P2.50mm_Vertical"
 			(at 45.72 101.6 0)
 			(hide yes)

Commit message: part numbers
Parts:
- C47, C48: LCSC C15849 -> -- mixed values --; LCSC P/N (none) -> C15849; Manufactuerer TAIYO YUDEN -> -- mixed values --; Mouser Part Number (none) -> -- mixed values --; P/N MLASU168SB5105KTNA01 -> CC0603KRX7R9BB105
- D21, D22: LCSC P/N (none) -> C6326606
- FAN1, FAN2: P/N (none) -> 105313-1104
- R82, R84: LCSC C25804 -> -- mixed values --; LCSC P/N (none) -> C25804; Manufactuerer Vishay -> -- mixed values --; P/N CRCW06035K10FKEC -> CR0603-FX-1002ELF
- R83, R87: LCSC P/N (none) -> C4216; P/N CRCW060310K0FKEI -> CRCW060333K0FKEA
- R85, R86: LCSC (none) -> -- mixed values --; LCSC P/N (none) -> C25804; Manufactuerer (none) -> -- mixed values --; P/N CRCW060310K0FKEI -> CR0603-FX-1002ELF
- U9: LCSC P/N (none) -> C621415

Commit message: fixed fan chip footprint and buck output capacitors
Parts:
- U9: footprint Package_DFN_QFN:QFN-16-1EP_1.8x2.6mm_P0.4mm_EP0.7x1.5mm -> Package_DFN_QFN:Texas_RGV0016A_VQFN-16-1EP_4x4mm_P0.65mm_EP2.1x2.1mm
Changed lines of the file:
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@@
 			)
 		)
-		(property "Footprint" "Package_DFN_QFN:QFN-16-1EP_1.8x2.6mm_P0.4mm_EP0.7x1.5mm"
+		(property "Footprint" "Package_DFN_QFN:Texas_RGV0016A_VQFN-16-1EP_4x4mm_P0.65mm_EP2.1x2.1mm"
 			(at 92.71 36.83 0)
 			(hide yes)
