File: hardware/HV_Minus_Contactor.kicad_sch (KiCad schematic)
At the start: 25 parts, among them J17 Contactor Connector, Q8 IRLML0030, Q9 IRLML0030, U8 DRV110APWR

Commit message: reviewed
Parts:
- TP9: now not fitted
Changed lines of the file:
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@@
 		(on_board yes)
 		(in_pos_files yes)
-		(dnp no)
+		(dnp yes)
 		(property "Reference" "TP9"
 			(at 118.11 71.755 0)

Commit message: part numbers
Parts:
- C41, C43: LCSC P/N (none) -> C105911; P/N (none) -> -- mixed values --
- C42: LCSC (none) -> -- mixed values --; LCSC P/N (none) -> C15849; Manufactuerer (none) -> -- mixed values --; Mouser Part Number (none) -> -- mixed values --; P/N (none) -> CC0603KRX7R9BB105
- C44: LCSC P/N (none) -> C14665; P/N (none) -> KGM15AR71C101KT
- C45: LCSC C15849 -> -- mixed values --; LCSC P/N (none) -> C15849; Manufactuerer (none) -> -- mixed values --; Mouser Part Number 963-UMK107BJ105KA-T -> -- mixed values --; P/N UMK107BJ105KA-T -> CC0603KRX7R9BB105
- C46: LCSC C14663 -> -- mixed values --; LCSC P/N (none) -> C14663; Mouser Part Number 963-HMK107B7104KA-T -> -- mixed values --; P/N HMK107B7104KA-T -> MLASH168SB7104KTNA01
- D18, D20: LCSC P/N (none) -> C6326606
- D19: LCSC P/N (none) -> C84263
- J17: P/N (none) -> 105313-1104
- Q8, Q9: LCSC P/N (none) -> C67272; P/N IRLML0030 -> IRLML0030TRPBF
- R72: LCSC P/N (none) -> C2933250; P/N (none) -> AC0603FR-0766K5L
- R73: LCSC P/N (none) -> C844719; P/N (none) -> CRCW06030000Z0EAHP
- R74, R79: LCSC (none) -> -- mixed values --; LCSC P/N (none) -> C21190; Manufactuerer (none) -> -- mixed values --; P/N (none) -> CRCW06031K00FKEI
- R75: LCSC P/N (none) -> C2906987; P/N (none) -> RK73B1JTTD124J
- R76, R80, R81: LCSC (none) -> -- mixed values --; LCSC P/N (none) -> C25804; Manufactuerer (none) -> -- mixed values --; P/N (none) -> CR0603-FX-1002ELF
- R77: LCSC P/N (none) -> C54920924; P/N (none) -> CR0603-FX-4301ELF
- R78: LCSC P/N (none) -> C2907004; P/N (none) -> RK73B1JTTD1R0J
- U8: P/N (none) -> DRV110APWR

Commit message: workday
Parts:
- renumbered J17 to J14, TP9 to TP8, TP10 to TP9
Changed lines of the file:
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@@
 		(in_pos_files yes)
 		(dnp no)
-		(property "Reference" "J17"
+		(property "Reference" "J14"
 			(at 250.825 33.6549 0)
 			(show_name no)
@@
 			(project "PS-BPSLeader"
 				(path "/d4a4ed4f-0983-4aef-b212-0e3284ab3963/3ea03975-64ac-45d5-b376-c81c9b8177bf"
-					(reference "J17")
+					(reference "J14")
 					(unit 1)
 				)
@@
 		(in_pos_files yes)
 		(dnp yes)
-		(property "Reference" "TP9"
+		(property "Reference" "TP8"
 			(at 118.11 71.755 0)
 			(show_name no)
@@
 			(project "PS-BPSLeader"
 				(path "/d4a4ed4f-0983-4aef-b212-0e3284ab3963/3ea03975-64ac-45d5-b376-c81c9b8177bf"
-					(reference "TP9")
+					(reference "TP8")
 					(unit 1)
 				)
@@
 		(in_pos_files yes)
 		(dnp yes)
-		(property "Reference" "TP10"
+		(property "Reference" "TP9"
 			(at 193.929 46.101 0)
 			(show_name no)
@@
 			(project "PS-BPSLeader"
 				(path "/d4a4ed4f-0983-4aef-b212-0e3284ab3963/3ea03975-64ac-45d5-b376-c81c9b8177bf"
-					(reference "TP10")
-					(unit 1)
-				)
+					(reference "TP9")
+					(unit 1)
+				)
