File: hardware/HV_Plus_Contactor.kicad_sch (KiCad schematic)
At the start: 25 parts, among them J16 Contactor Connector, Q6 IRLML0030, Q7 IRLML0030, U7 DRV110APWR

Commit message: reviewed
Parts:
- TP8: now not fitted
Changed lines of the file:
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@@
 		(on_board yes)
 		(in_pos_files yes)
-		(dnp no)
+		(dnp yes)
 		(property "Reference" "TP8"
 			(at 188.214 43.561 0)

Commit message: part numbers
Parts:
- C35, C37: LCSC P/N (none) -> C105911; P/N (none) -> -- mixed values --
- C36: LCSC (none) -> -- mixed values --; LCSC P/N (none) -> C15849; Manufactuerer (none) -> -- mixed values --; Mouser Part Number (none) -> -- mixed values --; P/N (none) -> CC0603KRX7R9BB105
- C38: LCSC P/N (none) -> C14665; P/N (none) -> KGM15AR71C101KT
- C39: LCSC C15849 -> -- mixed values --; LCSC P/N (none) -> C15849; Manufactuerer (none) -> -- mixed values --; Mouser Part Number 963-UMK107BJ105KA-T -> -- mixed values --; P/N UMK107BJ105KA-T -> CC0603KRX7R9BB105
- C40: LCSC C14663 -> -- mixed values --; LCSC P/N (none) -> C14663; Mouser Part Number 963-HMK107B7104KA-T -> -- mixed values --; P/N HMK107B7104KA-T -> MLASH168SB7104KTNA01
- D15, D17: LCSC P/N (none) -> C6326606
- D16: LCSC P/N (none) -> C84263
- J16: P/N (none) -> 105313-1104
- Q6, Q7: LCSC P/N (none) -> C67272; P/N IRLML0030 -> IRLML0030TRPBF
- R62: LCSC P/N (none) -> C2933250; P/N (none) -> AC0603FR-0766K5L
- R63: LCSC P/N (none) -> C844719; P/N (none) -> CRCW06030000Z0EAHP
- R64, R69: LCSC (none) -> -- mixed values --; LCSC P/N (none) -> C21190; Manufactuerer (none) -> -- mixed values --; P/N (none) -> CRCW06031K00FKEI
- R65: LCSC P/N (none) -> C2906987; P/N (none) -> RK73B1JTTD124J
- R66, R70, R71: LCSC (none) -> -- mixed values --; LCSC P/N (none) -> C25804; Manufactuerer (none) -> -- mixed values --; P/N (none) -> CR0603-FX-1002ELF
- R67: LCSC P/N (none) -> C54920924; P/N (none) -> CR0603-FX-4301ELF
- R68: LCSC P/N (none) -> C2907004; P/N (none) -> RK73B1JTTD1R0J
- U7: P/N (none) -> DRV110APWR

Commit message: workday
Parts:
- renumbered J16 to J13, TP7 to TP6, TP8 to TP7
Changed lines of the file:
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@@
 		(in_pos_files yes)
 		(dnp yes)
-		(property "Reference" "TP8"
+		(property "Reference" "TP7"
 			(at 188.214 43.561 0)
 			(show_name no)
@@
 			(project "PS-BPSLeader"
 				(path "/d4a4ed4f-0983-4aef-b212-0e3284ab3963/d0687915-3890-41dc-9a8f-e7ee1bda9492"
-					(reference "TP8")
+					(reference "TP7")
 					(unit 1)
 				)
@@
 		(in_pos_files yes)
 		(dnp yes)
-		(property "Reference" "TP7"
+		(property "Reference" "TP6"
 			(at 112.395 69.215 0)
 			(show_name no)
@@
 			(project "PS-BPSLeader"
 				(path "/d4a4ed4f-0983-4aef-b212-0e3284ab3963/d0687915-3890-41dc-9a8f-e7ee1bda9492"
-					(reference "TP7")
+					(reference "TP6")
 					(unit 1)
 				)
@@
 		(in_pos_files yes)
 		(dnp no)
-		(property "Reference" "J16"
+		(property "Reference" "J13"
 			(at 245.11 31.1149 0)
 			(show_name no)
@@
 			(project "PS-BPSLeader"
 				(path "/d4a4ed4f-0983-4aef-b212-0e3284ab3963/d0687915-3890-41dc-9a8f-e7ee1bda9492"
-					(reference "J16")
-					(unit 1)
-				)
+					(reference "J13")
+					(unit 1)
+				)
