File: hardware/Motor_Contactor.kicad_sch (KiCad schematic)
At the start: 25 parts, among them J15 Contactor Connector, Q4 IRLML0030, Q5 IRLML0030, U5 DRV110APWR

Commit message: reviewed
Parts:
- TP5: now not fitted
Changed lines of the file:
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@@
 		(on_board yes)
 		(in_pos_files yes)
-		(dnp no)
+		(dnp yes)
 		(property "Reference" "TP5"
 			(at 115.57 71.755 0)

Commit message: part numbers
Parts:
- C28, C30: LCSC P/N (none) -> C105911; P/N (none) -> -- mixed values --
- C29: LCSC (none) -> -- mixed values --; LCSC P/N (none) -> C15849; Manufactuerer (none) -> -- mixed values --; Mouser Part Number (none) -> -- mixed values --; P/N (none) -> CC0603KRX7R9BB105
- C31: LCSC P/N (none) -> C14665; P/N (none) -> KGM15AR71C101KT
- C32: LCSC C15849 -> -- mixed values --; LCSC P/N (none) -> C15849; Manufactuerer (none) -> -- mixed values --; Mouser Part Number 963-UMK107BJ105KA-T -> -- mixed values --; P/N UMK107BJ105KA-T -> CC0603KRX7R9BB105
- C33: LCSC C14663 -> -- mixed values --; LCSC P/N (none) -> C14663; Mouser Part Number 963-HMK107B7104KA-T -> -- mixed values --; P/N HMK107B7104KA-T -> MLASH168SB7104KTNA01
- D12, D14: LCSC P/N (none) -> C6326606
- D13: LCSC P/N (none) -> C84263
- J15: P/N (none) -> 105313-1104
- Q4, Q5: LCSC P/N (none) -> C67272; P/N IRLML0030 -> IRLML0030TRPBF
- R43: LCSC P/N (none) -> C2933250; P/N (none) -> AC0603FR-0766K5L
- R44: LCSC P/N (none) -> C844719; P/N (none) -> CRCW06030000Z0EAHP
- R45, R50: LCSC (none) -> -- mixed values --; LCSC P/N (none) -> C21190; Manufactuerer (none) -> -- mixed values --; P/N (none) -> CRCW06031K00FKEI
- R46: LCSC P/N (none) -> C2906987; P/N (none) -> RK73B1JTTD124J
- R47, R51, R52: LCSC (none) -> -- mixed values --; LCSC P/N (none) -> C25804; Manufactuerer (none) -> -- mixed values --; P/N (none) -> CR0603-FX-1002ELF
- R48: LCSC P/N (none) -> C54920924; P/N (none) -> CR0603-FX-4301ELF
- R49: LCSC P/N (none) -> C2907004; P/N (none) -> RK73B1JTTD1R0J
- U5: P/N (none) -> DRV110APWR

Commit message: workday
Parts:
- renumbered J15 to J12, TP5 to TP4, TP6 to TP5
Changed lines of the file:
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@@
 		(in_pos_files yes)
 		(dnp no)
-		(property "Reference" "J15"
+		(property "Reference" "J12"
 			(at 248.285 33.6549 0)
 			(show_name no)
@@
 			(project "PS-BPSLeader"
 				(path "/d4a4ed4f-0983-4aef-b212-0e3284ab3963/8dff3833-5b3d-484d-a711-1f7fb0d1bbda"
-					(reference "J15")
+					(reference "J12")
 					(unit 1)
 				)
@@
 		(in_pos_files yes)
 		(dnp yes)
-		(property "Reference" "TP5"
+		(property "Reference" "TP4"
 			(at 115.57 71.755 0)
 			(show_name no)
@@
 			(project "PS-BPSLeader"
 				(path "/d4a4ed4f-0983-4aef-b212-0e3284ab3963/8dff3833-5b3d-484d-a711-1f7fb0d1bbda"
-					(reference "TP5")
+					(reference "TP4")
 					(unit 1)
 				)
@@
 		(in_pos_files yes)
 		(dnp yes)
-		(property "Reference" "TP6"
+		(property "Reference" "TP5"
 			(at 191.389 46.101 0)
 			(show_name no)
@@
 			(project "PS-BPSLeader"
 				(path "/d4a4ed4f-0983-4aef-b212-0e3284ab3963/8dff3833-5b3d-484d-a711-1f7fb0d1bbda"
-					(reference "TP6")
-					(unit 1)
-				)
+					(reference "TP5")
+					(unit 1)
+				)
