File: hardware/PowerProtection.kicad_sch (KiCad schematic)
At the start: 18 parts, among them IC5 LM74502DDFR, Q13 PSMN012-100YS, Q14 PSMN012-100YS

Commit message: part numbers
Parts:
- C78: LCSC (none) -> -- mixed values --; Mouser Part Number (none) -> -- mixed values --
- C79: Mouser Part Number (none) -> -- mixed values --
- C81: LCSC P/N MSASH168SB5103KTNA01 -> C100042; P/N (none) -> CC0603KRX7R9BB103
- C82: Mouser P/N (none) -> -- mixed values --; Mouser Part Number (none) -> -- mixed values --; P/N GRM21BR61H106KE43K -> GRM21BR61H106KE43L
- C83, C84: LCSC (none) -> -- mixed values --; LCSC P/N (none) -> C14663; Mouser Part Number (none) -> -- mixed values --; P/N (none) -> MLASH168SB7104KTNA01
- D29: LCSC P/N (none) -> C183490; P/N (none) -> SMAF4758A-TP
- R119: Mouser Part Number 71-CRCW060310K0FKEI -> -- mixed values --; P/N CRCW060310K0FKEI -> CR0603-FX-1002ELF
- R121: P/N CRCW0603221KFKEA -> CRCW0603100KFKEE
- R123: P/N CRCW060310K0FKEI -> CRCW0603100KFKEE
Changed lines of the file:
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@@
 			)
 		)
-		(property "Description" "Unpolarized capacitor"
+		(property "Description" "-- mixed values --"
 			(at 129.54 90.17 0)
+			(hide yes)
+			(show_name no)
+			(do_not_autoplace no)
+			(effects
+				(font
+					(size 1.27 1.27)
+				)
+			)
+		)
+		(property "LCSC" "-- mixed values --"
+			(at 129.54 90.17 90)
+			(hide yes)
+			(show_name no)
+			(do_not_autoplace no)
+			(effects
+				(font
+					(size 1.27 1.27)
+				)
+			)
+		)
+		(property "LCSC P/N" "C14663"
+			(at 129.54 90.17 90)
+			(hide yes)
+			(show_name no)
+			(do_not_autoplace no)
+			(effects
+				(font
+					(size 1.27 1.27)
+				)
+			)
+		)
+		(property "Mouser Part Number" "-- mixed values --"
+			(at 129.54 90.17 90)
+			(hide yes)
+			(show_name no)
+			(do_not_autoplace no)
+			(effects
+				(font
+					(size 1.27 1.27)
+				)
+			)
+		)
+		(property "P/N" "MLASH168SB7104KTNA01"
+			(at 129.54 90.17 90)
 			(hide yes)
 			(show_name no)
@@
 		)
 		(property "Description" "Zener diode"
+			(at 43.18 83.82 0)
+			(hide yes)
+			(show_name no)
+			(do_not_autoplace no)
+			(effects
+				(font
+					(size 1.27 1.27)
+				)
+			)
+		)
+		(property "LCSC P/N" "C183490 "
+			(at 43.18 83.82 0)
+			(hide yes)
+			(show_name no)
+			(do_not_autoplace no)
+			(effects
+				(font
+					(size 1.27 1.27)
+				)
+			)
+		)
+		(property "P/N" "SMAF4758A-TP "
 			(at 43.18 83.82 0)
 			(hide yes)
@@
 			)
 		)
-		(property "Datasheet" ""
+		(property "Datasheet" "-- mixed values --"
 			(at 43.18 62.23 0)
 			(hide yes)
@@
 			)
 		)
-		(property "Description" "Resistor, US symbol"
+		(property "Description" "-- mixed values --"
 			(at 43.18 62.23 0)
 			(hide yes)
@@
 			)
 		)
-		(property "P/N" "CRCW060310K0FKEI"
+		(property "P/N" "CR0603-FX-1002ELF "
 			(at 43.18 62.23 0)
 			(hide yes)
@@
 			)
 		)
-		(property "Mouser Part Number" "71-CRCW060310K0FKEI"
+		(property "Mouser Part Number" "-- mixed values --"
 			(at 43.18 62.23 0)
 			(hide yes)
@@
 			)
 		)
-		(property "Description" "Unpolarized capacitor"
+		(property "Description" "-- mixed values --"
 			(at 34.29 50.8 0)
 			(hide yes)
@@
 		)
 		(property "LCSC P/N" "C14663"
+			(at 34.29 50.8 0)
+			(hide yes)
+			(show_name no)
+			(do_not_autoplace no)
+			(effects
+				(font
+					(size 1.27 1.27)
+				)
+			)
+		)
+		(property "LCSC" "-- mixed values --"
+			(at 34.29 50.8 0)
+			(hide yes)
+			(show_name no)
+			(do_not_autoplace no)
+			(effects
+				(font
+					(size 1.27 1.27)
+				)
+			)
+		)
+		(property "Mouser Part Number" "-- mixed values --"
 			(at 34.29 50.8 0)
 			(hide yes)
@@
 			)
 		)
-		(property "Description" "Unpolarized capacitor"
+		(property "Description" "-- mixed values --"
 			(at 110.49 90.17 0)
+			(hide yes)
+			(show_name no)
+			(do_not_autoplace no)
+			(effects
+				(font
+					(size 1.27 1.27)
+				)
+			)
+		)
+		(property "LCSC" "-- mixed values --"
+			(at 110.49 90.17 90)
+			(hide yes)
+			(show_name no)
+			(do_not_autoplace no)
+			(effects
+				(font
+					(size 1.27 1.27)
+				)
+			)
+		)
+		(property "LCSC P/N" "C14663"
+			(at 110.49 90.17 90)
+			(hide yes)
+			(show_name no)
+			(do_not_autoplace no)
+			(effects
+				(font
+					(size 1.27 1.27)
+				)
+			)
+		)
+		(property "Mouser Part Number" "-- mixed values --"
+			(at 110.49 90.17 90)
+			(hide yes)
+			(show_name no)
+			(do_not_autoplace no)
+			(effects
+				(font
+					(size 1.27 1.27)
+				)
+			)
+		)
+		(property "P/N" "MLASH168SB7104KTNA01"
+			(at 110.49 90.17 90)
 			(hide yes)
 			(show_name no)
@@
 			)
 		)
-		(property "LCSC P/N" "MSASH168SB5103KTNA01"
+		(property "LCSC P/N" "C100042 "
+			(at 60.96 63.5 0)
+			(hide yes)
+			(show_name no)
+			(do_not_autoplace no)
+			(effects
+				(font
+					(size 1.27 1.27)
+				)
+			)
+		)
+		(property "P/N" "CC0603KRX7R9BB103 "
 			(at 60.96 63.5 0)
 			(hide yes)
@@
 			)
 		)
-		(property "Description" "Unpolarized capacitor"
+		(property "Description" "-- mixed values --"
 			(at 109.22 50.8 0)
 			(hide yes)
@@
 			)
 		)
-		(property "P/N" "GRM21BR61H106KE43K"
+		(property "P/N" "GRM21BR61H106KE43L "
 			(at 109.22 53.975 0)
 			(hide yes)
@@
 		)
 		(property "LCSC P/N" "C440198"
+			(at 109.22 50.8 0)
+			(hide yes)
+			(show_name no)
+			(do_not_autoplace no)
+			(effects
+				(font
+					(size 1.27 1.27)
+				)
+			)
+		)
+		(property "Mouser P/N" "-- mixed values --"
+			(at 109.22 50.8 0)
+			(hide yes)
+			(show_name no)
+			(do_not_autoplace no)
+			(effects
+				(font
+					(size 1.27 1.27)
+				)
+			)
+		)
+		(property "Mouser Part Number" "-- mixed values --"
 			(at 109.22 50.8 0)
 			(hide yes)
@@
 			)
 		)
+		(property "Mouser Part Number" "-- mixed values --"
+			(at 35.56 83.82 0)
+			(hide yes)
+			(show_name no)
+			(do_not_autoplace no)
+			(effects
+				(font
+					(size 1.27 1.27)
+				)
+			)
+		)
 		(pin "2"
 		)
@@
 			)
 		)
-		(property "P/N" "CRCW0603221KFKEA"
+		(property "P/N" "CRCW0603100KFKEE  "
 			(at 115.57 77.47 0)
 			(hide yes)
@@
 			)
 		)
-		(property "P/N" "CRCW060310K0FKEI"
+		(property "P/N" "CRCW0603100KFKEE  "
 			(at 134.62 77.47 0)
 			(hide yes)

Commit message: workday
Parts:
- renumbered D28 to D30, D29 to D31
Changed lines of the file:
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@@
 		(in_pos_files yes)
 		(dnp no)
-		(property "Reference" "D29"
+		(property "Reference" "D31"
 			(at 40.64 82.296 0)
 			(show_name no)
@@
 			(project "PS-BPSLeader"
 				(path "/d4a4ed4f-0983-4aef-b212-0e3284ab3963/69244dac-f10b-499c-a2b2-3cdf1370aa1f/809e2845-19f2-4000-97b2-9d58cc5520c6"
-					(reference "D29")
+					(reference "D31")
 					(unit 1)
 				)
@@
 		(in_pos_files yes)
 		(dnp no)
-		(property "Reference" "D28"
+		(property "Reference" "D30"
 			(at 22.606 49.276 0)
 			(show_name no)
@@
 			(project "PS-BPSLeader"
 				(path "/d4a4ed4f-0983-4aef-b212-0e3284ab3963/69244dac-f10b-499c-a2b2-3cdf1370aa1f/809e2845-19f2-4000-97b2-9d58cc5520c6"
-					(reference "D28")
-					(unit 1)
-				)
+					(reference "D30")
+					(unit 1)
+				)
