File: hardware/Power_3V3_LDO.kicad_sch (KiCad schematic)
At the start: 5 parts, among them U16 MCP1826S

Commit message: part numbers
Parts:
- C89, C90: Mouser P/N GRM21BR61H106KE43K -> -- mixed values --; Mouser Part Number (none) -> -- mixed values --; P/N (none) -> GRM21BR61H106KE43L
Changed lines of the file:
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@@
 			)
 		)
-		(property "Description" "Unpolarized capacitor, small symbol"
-			(at 139.7 69.85 0)
-			(hide yes)
-			(show_name no)
-			(do_not_autoplace no)
-			(effects
-				(font
-					(size 1.27 1.27)
-				)
-			)
-		)
-		(property "Mouser P/N" "GRM21BR61H106KE43K"
+		(property "Description" "-- mixed values --"
+			(at 139.7 69.85 0)
+			(hide yes)
+			(show_name no)
+			(do_not_autoplace no)
+			(effects
+				(font
+					(size 1.27 1.27)
+				)
+			)
+		)
+		(property "Mouser P/N" "-- mixed values --"
 			(at 139.7 69.85 0)
 			(hide yes)
@@
 		)
 		(property "LCSC P/N" "C440198"
+			(at 139.7 69.85 0)
+			(hide yes)
+			(show_name no)
+			(do_not_autoplace no)
+			(effects
+				(font
+					(size 1.27 1.27)
+				)
+			)
+		)
+		(property "Mouser Part Number" "-- mixed values --"
+			(at 139.7 69.85 0)
+			(hide yes)
+			(show_name no)
+			(do_not_autoplace no)
+			(effects
+				(font
+					(size 1.27 1.27)
+				)
+			)
+		)
+		(property "P/N" "GRM21BR61H106KE43L "
 			(at 139.7 69.85 0)
 			(hide yes)
@@
 			)
 		)
-		(property "Description" "Unpolarized capacitor, small symbol"
-			(at 165.1 69.85 0)
-			(hide yes)
-			(show_name no)
-			(do_not_autoplace no)
-			(effects
-				(font
-					(size 1.27 1.27)
-				)
-			)
-		)
-		(property "Mouser P/N" "GRM21BR61H106KE43K"
+		(property "Description" "-- mixed values --"
+			(at 165.1 69.85 0)
+			(hide yes)
+			(show_name no)
+			(do_not_autoplace no)
+			(effects
+				(font
+					(size 1.27 1.27)
+				)
+			)
+		)
+		(property "Mouser P/N" "-- mixed values --"
 			(at 165.1 69.85 0)
 			(hide yes)
@@
 			(at 165.1 69.85 0)
 			(hide yes)
+			(show_name no)
+			(do_not_autoplace no)
+			(effects
+				(font
+					(size 1.27 1.27)
+				)
+			)
+		)
+		(property "Mouser Part Number" "-- mixed values --"
+			(at 165.1 69.85 0)
+			(hide yes)
+			(show_name no)
+			(do_not_autoplace no)
+			(effects
+				(font
+					(size 1.27 1.27)
+				)
+			)
+		)
+		(property "P/N" "GRM21BR61H106KE43L "
+			(at 165.1 69.85 0)
+			(hide yes)

Commit message: workday
Parts:
- renumbered D30 to D32
Changed lines of the file:
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@@
 		(dnp no)
 		(fields_autoplaced yes)
-		(property "Reference" "D30"
+		(property "Reference" "D32"
 			(at 133.604 57.15 0)
 			(show_name no)
@@
 			(project "PS-BPSLeader"
 				(path "/d4a4ed4f-0983-4aef-b212-0e3284ab3963/69244dac-f10b-499c-a2b2-3cdf1370aa1f/3ac4b541-f87d-4cd8-af8e-016705365d4a"
-					(reference "D30")
+					(reference "D32")
 					(unit 1)
 				)
