File: hardware/Power_USB_PD.kicad_sch (KiCad schematic)
At the start: 38 parts, among them IC3 CYPD3177-24LQXQ, Q10 SI7997DP-T1-GE3, Q11 SI7997DP-T1-GE3, Q12 IRLML0030

Commit message: reviewed
Parts:
- TP15, TP20: now not fitted
Changed lines of the file:
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@@
 		(on_board yes)
 		(in_pos_files yes)
-		(dnp no)
+		(dnp yes)
 		(property "Reference" "TP20"
 			(at 238.76 104.9019 0)
@@
 		(on_board yes)
 		(in_pos_files yes)
-		(dnp no)
+		(dnp yes)
 		(fields_autoplaced yes)
 		(property "Reference" "TP15"

Commit message: part numbers
Parts:
- C59: Mfg GRM21BR61H106KE43K -> -- mixed values --
- C66, C67, R100, R102, R99: Mfg (none) -> -- mixed values --
- R103, R98: P/N CRCW060349K9FKEC -> CR0603-FX-4992ELF
- R93, R94: Mfg CRCW06035K10FKEC -> -- mixed values --
- R97: Mouser Part Number (none) -> -- mixed values --; P/N CRCW060310K0FKEI -> CR0603-FX-1002ELF
Changed lines of the file:
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@@
 			)
 		)
-		(property "Datasheet" ""
+		(property "Datasheet" "-- mixed values --"
 			(at 44.45 55.88 0)
 			(hide yes)
@@
 			)
 		)
-		(property "Mfg" "GRM21BR61H106KE43K"
+		(property "Mfg" "-- mixed values --"
 			(at 44.45 55.88 0)
 			(hide yes)
@@
 			)
 		)
-		(property "Datasheet" ""
+		(property "Datasheet" "-- mixed values --"
 			(at 46.99 147.32 0)
 			(hide yes)
@@
 			)
 		)
-		(property "Description" "Resistor, small symbol"
+		(property "Description" "-- mixed values --"
 			(at 46.99 147.32 0)
 			(hide yes)
@@
 			)
 		)
-		(property "P/N" "CRCW060310K0FKEI "
+		(property "P/N" "CR0603-FX-1002ELF "
 			(at 46.99 147.32 0)
 			(hide yes)
@@
 			)
 		)
+		(property "Mouser Part Number" "-- mixed values --"
+			(at 46.99 147.32 0)
+			(hide yes)
+			(show_name no)
+			(do_not_autoplace no)
+			(effects
+				(font
+					(size 1.27 1.27)
+				)
+			)
+		)
 		(pin "2"
 		)
@@
 			)
 		)
-		(property "Datasheet" ""
+		(property "Datasheet" "-- mixed values --"
 			(at 40.64 95.25 0)
 			(hide yes)
@@
 			)
 		)
-		(property "Description" "Resistor"
+		(property "Description" "-- mixed values --"
 			(at 40.64 95.25 0)
 			(hide yes)
@@
 			)
 		)
-		(property "Mfg" "CRCW06035K10FKEC "
+		(property "Mfg" "-- mixed values --"
 			(at 40.64 95.25 0)
 			(hide yes)
@@
 			)
 		)
-		(property "Datasheet" ""
+		(property "Datasheet" "-- mixed values --"
 			(at 41.91 189.23 0)
 			(hide yes)
@@
 			)
 		)
-		(property "Description" "Resistor, small symbol"
+		(property "Description" "-- mixed values --"
 			(at 41.91 189.23 0)
 			(hide yes)
@@
 			)
 		)
-		(property "Datasheet" ""
+		(property "Datasheet" "-- mixed values --"
 			(at 81.28 62.23 0)
 			(hide yes)
@@
 			)
 		)
-		(property "Description" "Resistor, small symbol"
+		(property "Description" "-- mixed values --"
 			(at 81.28 62.23 0)
 			(hide yes)
@@
 			)
 		)
-		(property "Datasheet" ""
+		(property "Datasheet" "-- mixed values --"
 			(at 81.28 93.98 0)
 			(hide yes)
@@
 			)
 		)
-		(property "Description" "Resistor, small symbol"
+		(property "Description" "-- mixed values --"
 			(at 81.28 93.98 0)
 			(hide yes)
@@
 			)
 		)
+		(property "Mfg" "-- mixed values --"
+			(at 81.28 93.98 0)
+			(hide yes)
+			(show_name no)
+			(do_not_autoplace no)
+			(effects
+				(font
+					(size 1.27 1.27)
+				)
+			)
+		)
 		(pin "2"
 		)
@@
 			)
 		)
+		(property "Mfg" "-- mixed values --"
+			(at 248.92 49.53 0)
+			(hide yes)
+			(show_name no)
+			(do_not_autoplace no)
+			(effects
+				(font
+					(size 1.27 1.27)
+				)
+			)
+		)
 		(pin "2"
 		)
@@
 			)
 		)
-		(property "Datasheet" ""
+		(property "Datasheet" "-- mixed values --"
 			(at 74.93 58.42 0)
 			(hide yes)
@@
 			)
 		)
-		(property "Description" "Resistor, small symbol"
+		(property "Description" "-- mixed values --"
 			(at 74.93 58.42 0)
 			(hide yes)
@@
 			)
 		)
+		(property "Mfg" "-- mixed values --"
+			(at 74.93 58.42 90)
+			(hide yes)
+			(show_name no)
+			(do_not_autoplace no)
+			(effects
+				(font
+					(size 1.27 1.27)
+				)
+			)
+		)
 		(pin "2"
 		)
@@
 			)
 		)
-		(property "Datasheet" ""
+		(property "Datasheet" "-- mixed values --"
 			(at 41.91 156.21 0)
 			(hide yes)
@@
 			)
 		)
-		(property "Description" "Resistor, small symbol"
+		(property "Description" "-- mixed values --"
 			(at 41.91 156.21 0)
 			(hide yes)
@@
 			)
 		)
-		(property "Datasheet" ""
+		(property "Datasheet" "-- mixed values --"
 			(at 25.4 95.25 0)
 			(hide yes)
@@
 			)
 		)
-		(property "Description" "Resistor"
+		(property "Description" "-- mixed values --"
 			(at 25.4 95.25 0)
 			(hide yes)
@@
 			)
 		)
-		(property "Mfg" "CRCW06035K10FKEC "
+		(property "Mfg" "-- mixed values --"
 			(at 25.4 95.25 0)
 			(hide yes)
@@
 			)
 		)
-		(property "P/N" "CRCW060349K9FKEC"
+		(property "P/N" "CR0603-FX-4992ELF "
 			(at 46.99 180.34 0)
 			(hide yes)
@@
 			)
 		)
+		(property "Mfg" "-- mixed values --"
+			(at 259.08 49.53 0)
+			(hide yes)
+			(show_name no)
+			(do_not_autoplace no)
+			(effects
+				(font
+					(size 1.27 1.27)
+				)
+			)
+		)
 		(pin "2"
 		)
@@
 			)
 		)
-		(property "P/N" "CRCW060349K9FKEC"
+		(property "P/N" "CR0603-FX-4992ELF "
 			(at 88.9 147.32 0)
 			(hide yes)
@@
 			)
 		)
-		(property "Datasheet" ""
+		(property "Datasheet" "-- mixed values --"
 			(at 74.93 90.17 0)
 			(hide yes)
@@
 			)
 		)
-		(property "Description" "Resistor, small symbol"
+		(property "Description" "-- mixed values --"
 			(at 74.93 90.17 0)
 			(hide yes)
@@
 			(at 74.93 90.17 90)
 			(hide yes)
+			(show_name no)
+			(do_not_autoplace no)
+			(effects
+				(font
+					(size 1.27 1.27)
+				)
+			)
+		)
+		(property "Mfg" "-- mixed values --"
+			(at 74.93 90.17 90)
+			(hide yes)

Commit message: workday
Parts:
- renumbered D24 to D26, D25 to D27, D26 to D28, D27 to D29, TP15 to TP14, TP16 to TP15, TP17 to TP16, TP18 to TP17, TP19 to TP18, TP20 to TP19
Changed lines of the file:
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@@
 		(in_pos_files yes)
 		(dnp no)
-		(property "Reference" "D25"
+		(property "Reference" "D27"
 			(at 99.06 145.5419 90)
 			(show_name no)
@@
 			(project "PS-BPSLeader"
 				(path "/d4a4ed4f-0983-4aef-b212-0e3284ab3963/69244dac-f10b-499c-a2b2-3cdf1370aa1f/1b9256b7-8667-463d-8456-0ec3ca2120be"
-					(reference "D25")
+					(reference "D27")
 					(unit 1)
 				)
@@
 		(dnp no)
 		(fields_autoplaced yes)
-		(property "Reference" "#FLG07"
+		(property "Reference" "#FLG08"
 			(at 35.56 45.085 0)
 			(hide yes)
@@
 			(project "PS-BPSLeader"
 				(path "/d4a4ed4f-0983-4aef-b212-0e3284ab3963/69244dac-f10b-499c-a2b2-3cdf1370aa1f/1b9256b7-8667-463d-8456-0ec3ca2120be"
-					(reference "#FLG07")
+					(reference "#FLG08")
 					(unit 1)
 				)
@@
 		(in_pos_files yes)
 		(dnp yes)
-		(property "Reference" "TP20"
+		(property "Reference" "TP19"
 			(at 238.76 104.9019 0)
 			(hide yes)
@@
 			(project "PS-BPSLeader"
 				(path "/d4a4ed4f-0983-4aef-b212-0e3284ab3963/69244dac-f10b-499c-a2b2-3cdf1370aa1f/1b9256b7-8667-463d-8456-0ec3ca2120be"
-					(reference "TP20")
+					(reference "TP19")
 					(unit 1)
 				)
@@
 		(in_pos_files yes)
 		(dnp yes)
-		(property "Reference" "TP17"
+		(property "Reference" "TP16"
 			(at 135.89 169.4181 0)
 			(hide yes)
@@
 			(project "PS-BPSLeader"
 				(path "/d4a4ed4f-0983-4aef-b212-0e3284ab3963/69244dac-f10b-499c-a2b2-3cdf1370aa1f/1b9256b7-8667-463d-8456-0ec3ca2120be"
-					(reference "TP17")
+					(reference "TP16")
 					(unit 1)
 				)
@@
 		(in_pos_files yes)
 		(dnp no)
-		(property "Reference" "D24"
+		(property "Reference" "D26"
 			(at 38.862 54.102 90)
 			(show_name no)
@@
 			(project "PS-BPSLeader"
 				(path "/d4a4ed4f-0983-4aef-b212-0e3284ab3963/69244dac-f10b-499c-a2b2-3cdf1370aa1f/1b9256b7-8667-463d-8456-0ec3ca2120be"
-					(reference "D24")
+					(reference "D26")
 					(unit 1)
 				)
@@
 		(dnp no)
 		(fields_autoplaced yes)
-		(property "Reference" "D27"
+		(property "Reference" "D29"
 			(at 257.81 93.0274 90)
 			(show_name no)
@@
 			(project "PS-BPSLeader"
 				(path "/d4a4ed4f-0983-4aef-b212-0e3284ab3963/69244dac-f10b-499c-a2b2-3cdf1370aa1f/1b9256b7-8667-463d-8456-0ec3ca2120be"
-					(reference "D27")
+					(reference "D29")
 					(unit 1)
 				)
@@
 		(dnp no)
 		(fields_autoplaced yes)
-		(property "Reference" "#FLG011"
+		(property "Reference" "#FLG012"
 			(at 161.925 48.26 0)
 			(hide yes)
@@
 			(project "PS-BPSLeader"
 				(path "/d4a4ed4f-0983-4aef-b212-0e3284ab3963/69244dac-f10b-499c-a2b2-3cdf1370aa1f/1b9256b7-8667-463d-8456-0ec3ca2120be"
-					(reference "#FLG011")
+					(reference "#FLG012")
 					(unit 1)
 				)
@@
 		(dnp no)
 		(fields_autoplaced yes)
-		(property "Reference" "#FLG08"
+		(property "Reference" "#FLG09"
 			(at 35.56 67.945 0)
 			(hide yes)
@@
 			(project "PS-BPSLeader"
 				(path "/d4a4ed4f-0983-4aef-b212-0e3284ab3963/69244dac-f10b-499c-a2b2-3cdf1370aa1f/1b9256b7-8667-463d-8456-0ec3ca2120be"
-					(reference "#FLG08")
+					(reference "#FLG09")
 					(unit 1)
 				)
@@
 		(in_pos_files yes)
 		(dnp yes)
-		(property "Reference" "TP16"
+		(property "Reference" "TP15"
 			(at 135.89 136.3981 0)
 			(hide yes)
@@
 			(project "PS-BPSLeader"
 				(path "/d4a4ed4f-0983-4aef-b212-0e3284ab3963/69244dac-f10b-499c-a2b2-3cdf1370aa1f/1b9256b7-8667-463d-8456-0ec3ca2120be"
-					(reference "TP16")
+					(reference "TP15")
 					(unit 1)
 				)
@@
 		(in_pos_files yes)
 		(dnp no)
-		(property "Reference" "#FLG09"
+		(property "Reference" "#FLG010"
 			(at 129.54 169.545 0)
 			(hide yes)
@@
 			(project "PS-BPSLeader"
 				(path "/d4a4ed4f-0983-4aef-b212-0e3284ab3963/69244dac-f10b-499c-a2b2-3cdf1370aa1f/1b9256b7-8667-463d-8456-0ec3ca2120be"
-					(reference "#FLG09")
+					(reference "#FLG010")
 					(unit 1)
 				)
@@
 		(dnp yes)
 		(fields_autoplaced yes)
-		(property "Reference" "TP15"
+		(property "Reference" "TP14"
 			(at 41.91 44.9581 0)
 			(hide yes)
@@
 			(project "PS-BPSLeader"
 				(path "/d4a4ed4f-0983-4aef-b212-0e3284ab3963/69244dac-f10b-499c-a2b2-3cdf1370aa1f/1b9256b7-8667-463d-8456-0ec3ca2120be"
-					(reference "TP15")
+					(reference "TP14")
 					(unit 1)
 				)
@@
 		(in_pos_files yes)
 		(dnp yes)
-		(property "Reference" "TP19"
+		(property "Reference" "TP18"
 			(at 165.8619 45.72 0)
 			(hide yes)
@@
 			(project "PS-BPSLeader"
 				(path "/d4a4ed4f-0983-4aef-b212-0e3284ab3963/69244dac-f10b-499c-a2b2-3cdf1370aa1f/1b9256b7-8667-463d-8456-0ec3ca2120be"
-					(reference "TP19")
+					(reference "TP18")
 					(unit 1)
 				)
@@
 		(dnp no)
 		(fields_autoplaced yes)
-		(property "Reference" "#FLG010"
+		(property "Reference" "#FLG011"
 			(at 153.035 48.26 0)
 			(hide yes)
@@
 			(project "PS-BPSLeader"
 				(path "/d4a4ed4f-0983-4aef-b212-0e3284ab3963/69244dac-f10b-499c-a2b2-3cdf1370aa1f/1b9256b7-8667-463d-8456-0ec3ca2120be"
-					(reference "#FLG010")
+					(reference "#FLG011")
 					(unit 1)
 				)
@@
 		(in_pos_files yes)
 		(dnp yes)
-		(property "Reference" "TP18"
+		(property "Reference" "TP17"
 			(at 149.0981 50.8 0)
 			(hide yes)
@@
 			(project "PS-BPSLeader"
 				(path "/d4a4ed4f-0983-4aef-b212-0e3284ab3963/69244dac-f10b-499c-a2b2-3cdf1370aa1f/1b9256b7-8667-463d-8456-0ec3ca2120be"
-					(reference "TP18")
+					(reference "TP17")
 					(unit 1)
 				)
@@
 		(in_pos_files yes)
 		(dnp no)
-		(property "Reference" "D26"
+		(property "Reference" "D28"
 			(at 99.06 178.5619 90)
 			(show_name no)
@@
 			(project "PS-BPSLeader"
 				(path "/d4a4ed4f-0983-4aef-b212-0e3284ab3963/69244dac-f10b-499c-a2b2-3cdf1370aa1f/1b9256b7-8667-463d-8456-0ec3ca2120be"
-					(reference "D26")
+					(reference "D28")
 					(unit 1)
 				)
